File: atlas_hw/atlas.sch (KiCad schematic (older format))
At the start: 68 parts, among them J1 Micro_SD_Card_Det, J2 PSP_LCD, J3 PSP_TOUCH, J4 PSP_LCD_BL, Q1 Q_NMOS_DGS, SW1 SRST, SW2 PWR, U1 STM32H743VITx, U10 NCP600SNADJ, U11 STM6601CA2BDM6F, U12 TPS63050, U2 nRF52810-QCxx, U3 W957D8MFYA, U4 LSF0108, U5 LSF0108, U6 LSF0108, U7 NCP600SNADJ, U8 TLV62569DBV, U9 TPS61070, Y1 32MHz, Y2 32.768kHz

Commit message: Moved around STM6601 buttons
Parts:
- added D?: LOW_BAT, symbol Device:LED_Small_ALT
- added R?: 1k, symbol Device:R_Small
- SW1: value SRST -> SReset
- SW2: value PWR -> Power
Connections:
- wire segments 490 -> 493
Other:
- moved on the sheet: C12, C13, C14, C15, C16, C17, C18, C19, J1, J2, L6, L7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

Commit message: Added gps to sch and footprint work
Parts:
- added D2: 1PPS, symbol Device:LED_Small_ALT
- added D3: D_Schottky_x2_KCom_AAK, symbol Device:D_Schottky_x2_KCom_AAK
- added J5: DEBUG_STM, Connector_PinHeader_1.27mm:PinHeader_2x05_P1.27mm_Vertical_SMD, symbol atlas:Conn_ARM_JTAG_SWD_10
- added J6: DEBUG_NRF, Connector_PinHeader_1.27mm:PinHeader_2x05_P1.27mm_Vertical_SMD, symbol atlas:Conn_ARM_JTAG_SWD_10
- added Q2: Q_NMOS_DGS, symbol Device:Q_NMOS_DGS
- added R16, R17, R19, R20, R21, R23: NC, symbol Device:R_Small
- added R18: 0, symbol Device:R_Small
- added R22, R25: 1k, symbol Device:R_Small
- added R26, R27: 10k, symbol Device:R_Small
- added SW3: ResetSTM, symbol Switch:SW_Push
- added SW4: ResetNRF, symbol Switch:SW_Push
- added U13: Wurth_2613011037000, atlas:Elara-1, symbol atlas:Wurth_2613011037000
- added U14: MS5637, atlas:QFN-4_3x3_Pitch2mm, symbol atlas:MS5637
- gave numbers to parts that had none: 2
Connections:
- net labels added: GPS_ON_OFF, GPS_WAKEUP
- wire segments 493 -> 566
- no-connect marks 2 -> 5
Other:
- note added: "1.7-2.0V with 1.8V RAM"
- note removed: "1.7-2.0V with 1.8V RAM\n2.7-3.6V with 3.0V RAM"
- moved on the sheet: AE1, C1, C10, C11, C15, C16, C2, C3, C4, C5, C6, C7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

Commit message: sensors, touch, backlight-pwm
Parts:
- added C24, C25: 0.1u, symbol Device:C_Small
- added C26: 1u, symbol Device:C_Small
- added D4: D_Schottky_Small_ALT, symbol Device:D_Schottky_Small_ALT
- added L9: 3.9n, symbol Device:L_Small
- added Q3: Q_NMOS_DGS, symbol Device:Q_NMOS_DGS
- added R28, R31: 100k, symbol Device:R_Small
- added R29, R30, R32, R33: 4.7k, symbol Device:R_Small
- added R?: NC, symbol Device:R_Small
- added U15: PAM2841, Package_DFN_QFN:DFN-8-1EP_2x2mm_P0.5mm_EP0.9x1.5mm, symbol atlas:PAM2841
- added U16: MC6470, Package_LGA:LGA-12_2x2mm_P0.5mm, symbol atlas:MC6470
- U8: symbol Regulator_Switching:TLV62569DBV -> atlas-rescue:TLV62569DBV-Regulator_Switching
Connections:
- net labels added: MC6470_INTA, MC6470_INTM, STC911_INT_3V3, STC911_RESET, ~STC911_INT
- net labels removed: SPI2_MISO_SENSOR, SPI2_MOSI_SENSOR, SPI2_SCK_SENSOR
- wire segments 566 -> 646
- no-connect marks 5 -> 7
Other:
- moved on the sheet: AE1, C1, C10, C11, C2, C3, C4, C5, C6, C7, C8, C9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

Commit message: added charger, no 3.3v pin on mcu for usb
Parts:
- added C27, C30: 10u, symbol Device:C_Small
- added C28: 47n, symbol Device:C_Small
- added C29: 4.7u, symbol Device:C_Small
- added D5: CHARGER_STATUS, symbol Device:LED_Small_ALT
- added J10: AUX_THERM, symbol Connector_Generic:Conn_01x02
- added J7: USB_C_Receptacle_USB2.0, symbol Connector:USB_C_Receptacle_USB2.0
- added J8: CELL_THERM, symbol Connector_Generic:Conn_01x03
- added J9: CELL_BARE, symbol Connector_Generic:Conn_01x02
- added L10: 1u, symbol Device:L_Small
- added R34, R35: 5.1k, symbol Device:R_Small
- added R36, R37, R38, R39, R40, R45: 0, symbol Device:R_Small
- added R41, R42, R43: 100k, symbol Device:R_Small
- added R46, R47: NC, symbol Device:R_Small
- added U17: BQ25611D, Package_DFN_QFN:WQFN-24-1EP_4x4mm_P0.5mm_EP2.7x2.7mm_ThermalVias, symbol atlas:BQ25611D
- added U19: NX3L1T3157, Package_TO_SOT_SMD:SOT-886, symbol atlas:NX3L1T3157
- U9: value TPS61070 -> TPS61073
- gave numbers to parts that had none: 1
Connections:
- net labels added: BQ25611_INT, CELL_NEG, CELL_NTC, CELL_POS, USB_CHGR_D+, USB_CHGR_D-, USB_PORT_D+, USB_PORT_D-, USB_PORT_VBUS, USB_STM_D+, USB_STM_D-, VDD_SD_1V8
- net labels removed: USB_HS_D+, USB_HS_D-
- wire segments 646 -> 756
Other:
- note added: "Alternatively use AMUX, Remove Q1+R2."
- moved on the sheet: D2, J3, Q1, Q2, Q3, R17, R2, R22, R23, R25, R3, R31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

Commit message: stripped back, 3v3 ver with teseo
Parts:
- removed AE1: Antenna, symbol Device:Antenna
- removed C1, C20, C22, C23: 10u, symbol Device:C_Small
- removed C10, C11: 12p, symbol Device:C_Small
- removed C12, C14, C17, C19: C_Small, symbol Device:C_Small
- removed C2, C6: 0.1u, symbol Device:C_Small
- removed C21: 1n, symbol Device:C_Small
- removed C3: 100p, symbol Device:C_Small
- removed C4: 0.8p, symbol Device:C_Small
- removed C5: NC, symbol Device:C_Small
- removed C7, C8: 1p, symbol Device:C_Small
- removed C9: 2.2pF, symbol Device:C_Small
- removed D1: LOW_BAT, symbol Device:LED_Small_ALT
- removed D2: 1PPS, symbol Device:LED_Small_ALT
- removed L1, L3, L5: 3.9n, symbol Device:L_Small
- removed L2: 15u, symbol Device:L_Small
- removed L4: NC, symbol Device:L_Small
- removed L7, L8: L_Small, symbol Device:L_Small
- removed Q2, Q3: Q_NMOS_DGS, symbol Device:Q_NMOS_DGS
- removed R12, R13, R8: 200k, symbol Device:R_Small
- removed R14: 560k, symbol Device:R_Small
- removed R15: 180k, symbol Device:R_Small
- removed R17, R23, R44: NC, symbol Device:R_Small
- removed R22, R25: 1k, symbol Device:R_Small
- removed R31, R9: 100k, symbol Device:R_Small
- removed U10: NCP600SNADJ, Package_SO:TSOP-5_1.65x3.05mm_P0.95mm, symbol atlas:NCP600SNADJ
- removed U12: TPS63050, atlas:VQFN12_2.5x2.5_Pitch0.5mm, symbol atlas:TPS63050
- removed U13: Wurth_2613011037000, atlas:Elara-1, symbol atlas:Wurth_2613011037000
- removed U2: nRF52810-QCxx, Package_DFN_QFN:QFN-32-1EP_5x5mm_P0.5mm_EP3.6x3.6mm, symbol MCU_Nordic:nRF52810-QCxx
- removed U4, U5: LSF0108, Package_DFN_QFN:WQFN-20-1EP_2.5x4.5mm_P0.5mm_EP1x2.9mm, symbol atlas:LSF0108
- removed U8: TLV62569DBV, Package_TO_SOT_SMD:SOT-23-5, symbol atlas-rescue:TLV62569DBV-Regulator_Switching
- removed Y1: 32MHz, Crystal:Crystal_SMD_3225-4Pin_3.2x2.5mm, symbol Device:Crystal_Small
- removed Y2: 32.768kHz, Crystal:Crystal_SMD_3225-4Pin_3.2x2.5mm, symbol Device:Crystal_Small
- added AE?: 2088900001, symbol Device:Antenna
- added C? (x4): 22p, symbol Device:C_Small
- added C? (x4): NC, symbol Device:C_Small
- added C? (x2): 120p, symbol Device:C_Small
- added C? (x2): 1u, symbol Device:C_Small
- added C? (x2): C_Small, symbol Device:C_Small
- added D?: 1PPS, symbol Device:LED_Small_ALT
- added F?: B39162B8813P810, Filter:Filter_1109-5_1.1x0.9mm, symbol Filter:B39162B8813P810
- added L?: 5n6, symbol Device:L_Small
- added L?: L_Small, symbol Device:L_Small
- added Q?: Q_NMOS_DGS, symbol Device:Q_NMOS_DGS
- added R?: 1k, symbol Device:R_Small
- added R? (x4): 0, symbol Device:R_Small
- added R? (x3): 100k, symbol Device:R_Small
- added R? (x8): NC, symbol Device:R_Small
- added R?: 200k, symbol Device:R_Small
- added U?: QN9021, symbol atlas:QN9021
- added U?: BGA725L6, symbol atlas:BGA725L6
- added U?: Teseo-LIV3F, symbol atlas:Teseo-LIV3F
- added U?: MCP1811B, symbol atlas:MCP1811B
- added U?: TLV62569DBV, Package_TO_SOT_SMD:SOT-23-5, symbol atlas-rescue:TLV62569DBV-Regulator_Switching
- added Y? (x2): 32k, symbol Device:Crystal_Small
- added Y? (x2): 16M, symbol Device:Crystal_Small
- D3: value D_Schottky_x2_KCom_AAK -> DC
- J6: value DEBUG_NRF -> DEBUG_QN
- U1: value STM32H743VITx -> STM32H723VITx
- U3: value W957D8MFYA -> W957A8MFYA5I
Connections:
- net labels added: DEBUG_NRESET_QN, DEBUG_SWDCLK_QN, DEBUG_SWDIO_QN, GPS_1PPS, GPS_ANT_OFF, GPS_RESET, GPS_VCC_RF, SP4_MISO_QN, SP4_MOSI_QN, SP4_SCK_QN, STC911_INT, UART8_RX_QN, UART8_TX_QN, VCC_BACKUP, VCC_MCU_3V3, VCC_SYS
- net labels removed: DEBUG_NRESET_NRF, DEBUG_SWDCLK_NRF, DEBUG_SWDIO_NRF, DEC1, DEC2, DEC3, DEC4, GPS_ON_OFF, LCD_FFC_G4, LCD_FFC_G5, LCD_FFC_G6, LCD_FFC_G7, LCD_FFC_R4, LCD_FFC_R5, LCD_FFC_R6, LCD_FFC_R7, PWR_WKUP4_NRF, SP4_MISO_NRF, SP4_MOSI_NRF, SP4_SCK_NRF, STC911_INT_3V3, UART8_RX_NRF, UART8_TX_NRF, VCC_CELL_OUT, VCC_MCU_LV, VDD_SD_3V3, XC1_NRF, XC2_NRF, XL1_NRF, XL2_NRF, ~STC911_INT
- wire segments 756 -> 696
- no-connect marks 7 -> 6
Other:
- note added: "3.3V"
- note added: "Place to minimise bus capacitance."
- note removed: "1.7-2.0V with 1.8V RAM"
- note removed: "2.3-3.6V"
- moved on the sheet: C13, C15, C16, C18, C24, C25, C26, C27, C28, C29, C30, D3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

Commit message: push to pcb
Parts:
- removed C? (x2): NC, symbol Device:C_Small
- removed J7: USB_C_Receptacle_USB2.0, symbol Connector:USB_C_Receptacle_USB2.0
- removed R32: 4.7k, symbol Device:R_Small
- removed R35: 5.1k, symbol Device:R_Small
- removed R43: 100k, symbol Device:R_Small
- removed U?: QN9021, symbol atlas:QN9021
- removed Y?: 16M, symbol Device:Crystal_Small
- added AE1: CHIP, symbol Device:Antenna
- added C11, C16, C22, C23, C24, C25, C26, C28, C29, C30, C32, C33, C34, C35, C38, C39, C45, C54, C55, C56, C57, C58, C59, C6, C60, C61, C9: 0.1u, symbol Device:C_Small
- added C12: 100p, symbol Device:C_Small
- added C14, C17, C18: 1p, symbol Device:C_Small
- added C15: NP, symbol Device:C_Small
- added C20: 2.2p, symbol Device:C_Small
- added C27, C31: 1u, symbol Device:C_Small
- added C5: 10u, symbol Device:C_Small
- added C51: 4.7uu, symbol Device:C_Small
- added C53: 2.2u, symbol Device:C_Small
- added D2: STM_STATUS, symbol Device:LED_Small_ALT
- added D3: NRF_STATUS, symbol Device:LED_Small_ALT
- added D7: USB_DETECT, symbol Device:LED_Small_ALT
- added J1: USB_C_Receptacle_USB2.0, Connector_USB:USB_C_Receptacle_Amphenol_12401548E4-2A, symbol Connector:USB_C_Receptacle_USB2.0
- added L1, L4, L6: 3.9n, symbol Device:L_Small
- added L2: 15u, symbol Device:L_Small
- added L5: NP, symbol Device:L_Small
- added Q2, Q3, Q5: Q_NMOS_DGS, Package_TO_SOT_SMD:SOT-23, symbol Device:Q_NMOS_DGS
- added R10, R11, R87: 1k, symbol Device:R_Small
- added R12, R13: 5.1k, symbol Device:R_Small
- added R14, R15, R16, R17, R44, R46, R80, R81, R88, R89: 0, symbol Device:R_Small
- added R28, R29, R41, R42, R58, R59, R60, R61, R62, R63, R64, R65, R66, R67, R68, R69, R70, R71, R72, R73, R74: NP, symbol Device:R_Small
- added R7, R8, R85, R86: 100k, symbol Device:R_Small
- added U5: nRF52810-QCxx, Package_DFN_QFN:QFN-32-1EP_5x5mm_P0.5mm_EP3.6x3.6mm, symbol MCU_Nordic:nRF52810-QCxx
- added U6: LC709203F, atlas:WDFN-8_3x4mm_0.6mm_1.96x2.56mm, symbol atlas:LC709203F
- added Y3: 32M, symbol Device:Crystal_Small
- C1, C3: renamed from C?; value NC -> NP
- C13, C7: renamed from C?; value C_Small -> 1u
- C2, C4: renamed from C?; value 22p -> 12p
- C48: renamed from C24; value 0.1u -> 1u
- D1: renamed from D?; value 1PPS -> GPS_1PPS
- D5: value CHARGER_STATUS -> CHARGE_STATUS
- J4: renamed from J6; value DEBUG_QN -> DEBUG_NRF
- Q1: renamed from Q?; footprint (none) -> Package_TO_SOT_SMD:SOT-23
- Q4: renamed from Q1; footprint (none) -> Package_TO_SOT_SMD:SOT-23
- R18: renamed from R16; value NC -> NP
- R20: renamed from R19; value NC -> NP
- R21: renamed from R20; value NC -> NP
- R22: renamed from R21; value NC -> NP
- R26, R27, R48, R49, R50, R51, R52, R53: renamed from R?; value NC -> NP
- R33: value 4.7k -> 100k
- R34: value 5.1k -> 100k
- R36, R38, R39: value 0 -> 100k
- R37: value 0 -> 1k
- R45: renamed from R46; value NC -> NP
- R56: renamed from R10; value NC -> NP
- R57: renamed from R11; value NC -> NP
- R77: renamed from R47; value NC -> NP
- R82: renamed from R5; value NC -> NP
- U12: renamed from U?; footprint (none) -> atlas:TSLP-6-2
- U14: renamed from U7; value NCP600SNADJ -> NPP600SNADJ
- U3: renamed from U?; footprint (none) -> Package_TO_SOT_SMD:SOT-23
- U7: renamed from U?; footprint (none) -> RF_Module:ublox_MAX
- gave numbers to parts that had none: 23
- renumbered C27 to C36, C15 to C37, C16 to C40, C28 to C41, C29 to C42, C30 to C44, C13 to C47, C25 to C49, C18 to C50, C26 to C52, D3 to D4, D4 to D6, J2 to J10, J5 to J2, J8 to J5, J9 to J6, J10 to J7, J1 to J8, J4 to J9, L9 to L10, L10 to L7, L6 to L9, R18 to R19, R40 to R24, R26 to R25, R27 to R30, R41 to R31, R42 to R32, R24 to R35, R45 to R43, R28 to R47, R2 to R54, R1 to R55, R3 to R75, R4 to R76, R29 to R78, R30 to R79, R6 to R83, R7 to R84, U17 to U10, U6 to U13, U9 to U15, U15 to U16, U19 to U17, U3 to U2, U14 to U8, U16 to U9
Connections:
- net LCD_FFC_B4 is gone; now on net LTDC_B4: J10.21 (Pin_21), J10.25 (Pin_25)
- net LCD_FFC_B5 is gone; now on net LTDC_B5: J10.22 (Pin_22), J10.26 (Pin_26)
- net LCD_FFC_B6 is gone; now on net LTDC_B6: J10.23 (Pin_23), J10.27 (Pin_27)
- net LCD_FFC_B7 is gone; now on net LTDC_B7: J10.24 (Pin_24), J10.28 (Pin_28)
- net LCD_FFC_DE is gone; now on net LTDC_DE: J10.31 (Pin_31)
- net LTDC_CLK is gone; now on net LTDC_CK: U1.44 (PE14)
- net LTDC_HSYNC is gone; now on net LTDC_HS: U1.63 (PC6)
- net LTDC_VSYNC is gone; now on net LTDC_VS: U1.28 (PA4)
- net PWR_WKIP1_ONOFF is gone; now on net STC911_INT: U1.22 (PA0)
- net VCC_LCD_IO is gone; now on net VCC_MCU_3V3: J3.4 (Pin_4)
- net BQ25611_INT: now also U1.7 (PC13), U10.7 (~INT); no longer U1.52 (PB13)
- net CELL_POS: now also C31.2, U6.3 (VDD)
- net EN_MCU_PWR: now also R41.2, R42.1
- net GND: now also F1.3, U10.17 (GND), U10.18 (GND), U10.25 (GND), U10.9 (~CE), U7.1 (GND), U7.12 (GND_RF), C11.2, C12.1, C14.1, C15.1, C16.1, C17.1, C18.1, C22.2, C23.2, C24.2, C25.2, C26.2, C27.2, C28.2, C29.2, C30.2, C31.1, C32.2, C33.2, C34.2, C35.2, C38.2, C39.2, C45.1, C5.1, C51.2, C53.2, C54.2, C55.2, C56.1, C57.1, C58.1, C59.2, C6.2, C60.2, C61.2, C9.1, J1.A1 (GND), J1.A12 (GND), J1.B1 (GND), J1.B12 (GND), J1.S1 (SHIELD), L5.2, Q2.3 (S), Q3.3 (S), Q5.3 (S), R12.1, R13.2, R42.2, R58.1, R59.1, R60.1, R61.1, R62.1, R63.1, R64.1, R65.1, R66.1, R67.1, R68.1, R69.1, R7.2, R70.1, R71.1, R72.1, R73.1, R8.2, R85.2, R87.2, R88.2, R89.2, U5.20 (VSS), U5.29 (VSS), U5.33 (VSS), U6.1 (TEST), U6.2 (VSS); no longer R34.1, U13.18 (B0), U13.3 (A0)
- net GPS_1PPS: now also U7.4 (1PPS)
- net GPS_ANT_OFF: now also U7.13 (Ant_OFF)
- net GPS_RESET: now also U7.9 (~SRST)
- net GPS_VCC_RF: now also U7.14 (VCC_RF), C45.2
- net GPS_WAKEUP: now also U7.5 (WAKEUP)
- net I2C1_SCL_SYSTEM: now also J3.2 (Pin_2), U1.93 (PB7), U10.5 (SCL), U10.6 (SDA), U6.7 (SDA), U6.8 (SCL); no longer U10.9 (~CE)
- net I2C_SCL_SENSOR: now also U7.17 (SCL), R28.2; no longer R33.1, U8.2 (SDA), U9.2 (SDA)
- net I2C_SDA_SENSOR: now also U7.16 (SDA), U8.2 (SDA), U9.2 (SDA), R29.2
- net LPUART1_RX_GPS: now also U7.3 (RX)
- net LPUART1_TX_GPS: now also U7.2 (TX)
- net LTDC_B4: now also R66.2
- net LTDC_B5: now also R67.2
- net LTDC_B6: now also R68.2
- net LTDC_B7: now also R69.2
- net LTDC_DE: now also R71.2
- net LTDC_G4: now also R62.2
- net LTDC_G5: now also R63.2
- net LTDC_G6: now also R64.2
- net LTDC_G7: now also R65.2
- net LTDC_R4: now also R58.2
- net LTDC_R5: now also R59.2
- net LTDC_R6: now also R60.2
- net LTDC_R7: now also R61.2
- net MC6470_INTA: now also R34.2
- net MC6470_INTM: now also R38.2
- net PWR_BTN_OUT: now also R39.2, U1.87 (PD6); no longer U1.88 (PD7)
- net PWR_MCU_INT: now also R33.2, U1.88 (PD7), U5.26 (P0.25); no longer U1.87 (PD6)
- net PWR_MCU_NRST: now also R36.2
- net USB_CHGR_D+: now also R17.1; no longer R39.1
- net USB_CHGR_D-: now also R16.1; no longer R38.1
- net USB_PORT_D+: now also J1.A6 (D+), J1.B6 (D+), R15.2, R17.2; no longer R37.2, R39.2
- net USB_PORT_D-: now also J1.A7 (D-), J1.B7 (D-), R14.2, R16.2; no longer R36.2, R38.2
- net USB_PORT_VBUS: now also C27.1, C35.1, D7.2 (A), J1.A4 (VBUS), J1.A9 (VBUS), J1.B4 (VBUS), J1.B9 (VBUS), Q5.2 (G), R85.1
- net USB_STM_D+: now also R15.1; no longer R37.1
- net USB_STM_D-: now also R14.1; no longer R36.1
- net VCC_BACKUP: now also U7.6 (VBAT), C30.1
- net VCC_LCD_PWR: now also R80.2; no longer J10.35 (Pin_35), J10.36 (Pin_36)
- net VCC_MCU_3V3: now also R33.1, R34.1, R36.1, R38.1, R39.1, U7.7 (VCCIO), U7.8 (VCC), C22.1, C23.1, C24.1, C25.1, C26.1, C28.1, C29.1, C32.1, C33.1, C34.1, C38.1, C56.2, C57.2, C58.2, C59.1, C61.1, C9.2, D2.2 (A), D3.2 (A), R28.1, R29.1, R44.1, R81.2, R86.1, U5.25 (VDD), U5.32 (VDD), U5.9 (VDD); no longer J10.3 (Pin_3), J10.4 (Pin_4), R33.2, U14.1 (IN)
- net VCC_SYS: now also C44.2, D5.2 (A), L7.2, U10.15 (SYS), U10.16 (SYS), C39.1, R41.1, R46.2; no longer C48.2, L10.1, U16.1 (VIN)
- net VDD_SD_1V8: now also R74.2; no longer R75.2, R77.2
- net VDD_SD_IO_3V3_1V8: now also C60.1
- net BTN_ENTER: now reaches U1.16 (PC1)
- net NRF_INT: now reaches U1.2 (PE3)
- net NRF_INT: now also U5.8 (P0.10)
- net at R3.2, U1.21 (VDDA): now also C11.1
- net LC709203_INT: now reaches U1.23 (PA1)
- net LC709203_INT: now also U6.4 (ALARM)
- net ~USB_DET: now reaches U1.3 (PE4)
- net ~USB_DET: now also Q5.1 (D), R86.2
- net at R1.1, U1.6 (VBAT): now also C6.1
- net CHG_STAT: now reaches U10.4 (STAT)
- net CHG_STAT: now also R37.1
- net XL2_NRF: now reaches C4.2, Y2.2
- net XL2_NRF: now also U5.3 (P0.01/XL2)
- net XL1_NRF: now reaches C2.2, Y2.1
- net XL1_NRF: now also U5.2 (P0.00/XL1)
- net at C43.2: now also U7.10 (RF_IN)
- net at D5.1 (K): now also R37.2
- net DEBUG_NRESET_QN renamed DEBUG_NRESET_NRF
- net DEBUG_NRESET_NRF: now also U5.16 (P0.21/~RESET)
- net DEBUG_SWDCLK_QN renamed DEBUG_SWDCLK_NRF
- net DEBUG_SWDCLK_NRF: now also U5.17 (SWDCLK)
- net DEBUG_SWDIO_QN renamed DEBUG_SWDIO_NRF
- net DEBUG_SWDIO_NRF: now also U5.18 (SWDIO)
- removed net I2C1_SDA_SYSTEM: J3.2 (Pin_2), U1.93 (PB7), U10.7 (~INT)
- net LCD_FFC_CK renamed LTDC_CK
- net LTDC_CK: now also R70.2
- net LCD_FFC_HS renamed LTDC_HS
- net LTDC_HS: now also R72.2
- net LCD_FFC_VS renamed LTDC_VS
- net LTDC_VS: now also R73.2
- net LED_STATUS renamed STM_STATUS
- net STM_STATUS: now also Q2.2 (G), R7.1
- net OCTOSPIM_P1_NCLK renamed OCTOSPIM_P1_NPLK
- net OCTOSPIM_P1_NCS renamed OCTOSPIM_P1_NPS
- net SP4_MISO_QN renamed SP4_MISO_NRF
- net SP4_MISO_NRF: now also U5.11 (P0.14)
- net SP4_MOSI_QN renamed SP4_MOSI_NRF
- net SP4_MOSI_NRF: now also U5.10 (P0.12)
- net SP4_SCK_QN renamed SP4_SCK_NRF
- net SP4_SCK_NRF: now also U5.12 (P0.15)
- net UART8_RX_QN renamed UART8_RX_NRF
- net UART8_RX_NRF: now also U5.13 (P0.16)
- net UART8_TX_QN renamed UART8_TX_NRF
- net UART8_TX_NRF: now also U5.14 (P0.18)
- new net: C14.2, L4.1, U5.19 (ANT)
- new net: C17.2, U5.23 (XC1), Y3.2
- new net: C18.2, U5.24 (XC2), Y3.1
- new net: L2.2, U5.31 (DCC)
- new net: C54.1, C55.1, J10.3 (Pin_3), J10.4 (Pin_4), R81.1
- new net: C51.1, C53.1, J10.35 (Pin_35), R80.1
- new net: R74.1, R75.2, R77.2
- new net: R44.2, U14.1 (IN)
- new net: R89.1, U13.18 (B0)
- new net: R88.1, U13.3 (A0)
- new net: C20.2, L4.2
- new net: C20.1, L5.1, L6.1
- new net: AE1.1 (A), L6.2
- new net: L1.2, L2.1
- new net: C48.2, L10.1, R46.1, U16.1 (VIN)
- new net: D2.1 (K), R10.1
- new net: Q2.1 (D), R10.2
- new net: D3.1 (K), R11.1
- new net: Q3.1 (D), R11.2
- new net: J1.A5 (CC1), R12.2
- new net: J1.B5 (CC2), R13.1
- new net: D7.1 (K), R87.1
- new net DEC1: C12.2, U5.1 (DEC1)
- new net DEC2: C15.2, U5.21 (DEC2)
- new net DEC3: C16.2, U5.22 (DEC3)
- new net DEC4: C5.2, L1.1, U5.30 (DEC4)
- new net NRF_STATUS: Q3.2 (G), R8.1, U5.15 (P0.20)
Other:
- note added: "NPP600 should maintain low Iq in dropout."
- note added: "Place to minimise bus capacitaNPe."
- note removed: "NCP600 should maintain low Iq in dropout."
- note removed: "Place to minimise bus capacitance."
- moved on the sheet: AE2, C10, C13, C19, C2, C21, C36, C37, C4, C40, C41, C42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

Commit message: Added additional passives, assigned fp
Parts:
- removed R58, R59, R60, R61, R62, R63, R64, R65, R66, R67, R68, R69, R70, R71, R72, R73: NP, symbol Device:R_Small
- added C62, C63: 1u, Capacitor_SMD:C_0402_1005Metric, symbol Device:C_Small
- added RN1, RN2, RN3, RN4: R_Pack04, Resistor_SMD:R_Array_Concave_4x0402, symbol Device:R_Pack04
- AE1: footprint (none) -> Resistor_SMD:R_1206_3216Metric
- AE2: footprint (none) -> atlas:2088900001
- C1, C11, C12, C14, C15, C16, C17, C18, C19, C2, C20, C21, C22, C23, C24, C25, C26, C28, C29, C3, C30, C32, C33, C34, C35, C37, C38, C39, C4, C40, C41, C43, C45, C46, C49, C54, C55, C56, C57, C58, C59, C6, C60, C61, C9: footprint (none) -> Capacitor_SMD:C_0402_1005Metric
- C10, C13, C27, C31, C48, C52, C7, C8: footprint (none) -> Capacitor_SMD:C_0603_1608Metric
- C36, C44, C5: footprint (none) -> Capacitor_SMD:C_0805_2012Metric
- C42: value 4.7u -> 10u; footprint (none) -> Capacitor_SMD:C_0805_2012Metric
- C47, C50: value C_Small -> 1u; footprint (none) -> Capacitor_SMD:C_0603_1608Metric
- C51: value 4.7uu -> 10u; footprint (none) -> Capacitor_SMD:C_0805_2012Metric
- C53: value 2.2u -> 1u; footprint (none) -> Capacitor_SMD:C_0603_1608Metric
- D1, D2, D3, D5, D7: footprint (none) -> LED_SMD:LED_0805_2012Metric
- D4: footprint (none) -> Package_TO_SOT_SMD:SOT-23
- D6: footprint (none) -> Diode_SMD:D_SOD-123F
- J3: footprint (none) -> Connector_FFC-FPC:Hirose_FH12-6S-0.5SH_1x06-1MP_P0.50mm_Horizontal
- J5: footprint (none) -> Connector_JST:JST_GH_SM03B-GHS-TB_1x03-1MP_P1.25mm_Horizontal
- J6, J7: footprint (none) -> Connector_JST:JST_GH_SM02B-GHS-TB_1x02-1MP_P1.25mm_Horizontal
- J9: footprint (none) -> atlas:Kyocera_046298_004_1x04_P0.5mm_Bottom
- L1, L8: footprint (none) -> Inductor_SMD:L_0603_1608Metric
- L10, L2, L3, L7, L9: footprint (none) -> Inductor_SMD:L_6.3x6.3_H3
- L4, L5, L6: footprint (none) -> Inductor_SMD:L_0402_1005Metric
- R1, R10, R11, R12, R13, R14, R15, R16, R17, R18, R19, R2, R20, R21, R22, R23, R24, R25, R26, R27, R28, R29, R3, R30, R31, R32, R33, R34, R35, R36, R37, R38, R39, R4, R40, R41, R42, R43, R44, R45, R46, R47, R48, R49, R5, R50, R51, R52, R53, R54, R55, R56, R57, R6, R7, R74, R75, R76, R77, R78, R79, R8, R80, R81, R82, R83, R84, R85, R86, R87, R88, R89, R9: footprint (none) -> Resistor_SMD:R_0402_1005Metric
- SW1, SW2, SW3, SW4: footprint (none) -> Button_Switch_SMD:SW_SPST_B3U-1000P
- Y1, Y3: footprint (none) -> Crystal:Crystal_SMD_2016-4Pin_2.0x1.6mm
- Y2, Y4: footprint (none) -> Crystal:Crystal_SMD_2012-2Pin_2.0x1.2mm
Connections:
- net GND: now also C62.2, C63.2, RN1.1 (R1.1), RN1.2 (R2.1), RN1.3 (R3.1), RN1.4 (R4.1), RN2.1 (R1.1), RN2.2 (R2.1), RN2.3 (R3.1), RN2.4 (R4.1), RN3.1 (R1.1), RN3.2 (R2.1), RN3.3 (R3.1), RN3.4 (R4.1), RN4.1 (R1.1), RN4.2 (R2.1), RN4.3 (R3.1), RN4.4 (R4.1)
- net LTDC_B4: now also RN3.8 (R1.2)
- net LTDC_B5: now also RN3.7 (R2.2)
- net LTDC_B6: now also RN3.6 (R3.2)
- net LTDC_B7: now also RN3.5 (R4.2)
- net LTDC_CK: now also RN4.8 (R1.2)
- net LTDC_DE: now also RN4.7 (R2.2)
- net LTDC_G4: now also RN2.8 (R1.2)
- net LTDC_G5: now also RN2.7 (R2.2)
- net LTDC_G6: now also RN2.6 (R3.2)
- net LTDC_G7: now also RN2.5 (R4.2)
- net LTDC_HS: now also RN4.6 (R3.2)
- net LTDC_R4: now also RN1.8 (R1.2)
- net LTDC_R5: now also RN1.7 (R2.2)
- net LTDC_R6: now also RN1.6 (R3.2)
- net LTDC_R7: now also RN1.5 (R4.2)
- net LTDC_VS: now also RN4.5 (R4.2)
- net VDD_SD_1V8: now also C63.1
- net at R44.2, U14.1 (IN): now also C62.1
Other:
- moved on the sheet: C51, C53, C56, C57, C58, Q4, R43, R44, R45, R54, R75, R76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

Commit message: started layout
Parts:
- removed R45, R48, R49, R50, R51, R52, R53: NP, Resistor_SMD:R_0402_1005Metric, symbol Device:R_Small
- removed U12: BGA725L6, atlas:TSLP-6-2, symbol atlas:BGA725L6
- removed U17: NX3L1T3157, Package_TO_SOT_SMD:SOT-886, symbol atlas:NX3L1T3157
- added RN5, RN6: R_Pack04, Resistor_SMD:R_Array_Concave_4x0402, symbol Device:R_Pack04
- added U12: BGU7007, atlas:6-XSON_1.5x1.0mm_0.5mm, symbol atlas:BGU7007
- Y1, Y3: footprint Crystal:Crystal_SMD_2016-4Pin_2.0x1.6mm -> Crystal:Crystal_SMD_3225-4Pin_3.2x2.5mm
- Y2, Y4: footprint Crystal:Crystal_SMD_2012-2Pin_2.0x1.2mm -> Crystal:Crystal_SMD_3225-4Pin_3.2x2.5mm
Connections:
- net GND: now also RN6.3 (R3.1), RN6.4 (R4.1), RN6.5 (R4.2), RN6.6 (R3.2), U12.1 (G), U12.2 (G)
- net GPS_ANT_OFF: now also U12.5
- net GPS_VCC_RF: now also U12.4 (VCC)
- net SDMMC1_CK: now also RN5.4 (R4.1)
- net SDMMC1_CMD: now also RN5.3 (R3.1)
- net SDMMC1_D0: now also RN6.1 (R1.1)
- net SDMMC1_D1: now also RN6.2 (R2.1)
- net SDMMC1_D2: now also RN5.1 (R1.1)
- net SDMMC1_D3: now also RN5.2 (R2.1)
- net SD_CLK: now also RN5.5 (R4.2)
- net SD_CMD: now also RN5.6 (R3.2)
- net SD_D0: now also RN6.8 (R1.2)
- net SD_D1: now also RN6.7 (R2.2)
- net SD_D2: now also RN5.8 (R1.2)
- net SD_D3: now also RN5.7 (R2.2)
- net at F1.1: now also U12.6
- net at L8.1: now also U12.3
Other:
- note added: "Place under U13"
- note removed: "Alternatively use AMUX, Remove Q1+R2."
- note removed: "Place to minimise bus capacitaNPe."
- moved on the sheet: C35, C36, C41, C42, C44, C59, C60, C61, C62, C63, D5, J5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
