File: atlas_hw/atlas.sch (KiCad schematic (older format))
At the start: 192 parts, among them J1 USB_C_Receptacle_USB2.0, J10 PSP_LCD, J2 DEBUG_STM, J3 PSP_TOUCH, J4 DEBUG_NRF, J5 CELL_THERM, J8 Micro_SD_Card_Det, J9 PSP_LCD_BL, Q1 Q_NMOS_DGS, Q2 Q_NMOS_DGS, Q3 Q_NMOS_DGS, Q4 Q_NMOS_DGS, Q5 Q_NMOS_DGS, SW1 SReset, SW2 Power, SW3 ResetSTM, SW4 ResetNRF, U1 STM32H723VITx, U10 BQ25611D, U11 STM6601CA2BDM6F, U12 BGU7007, U13 LSF0108, U14 NPP600SNADJ, U15 TPS61073, U16 PAM2841, U2 W957A8MFYA5I, U3 MCP1811B, U4 TLV62569DBV, U5 nRF52810-QCxx, U6 LC709203F, U7 Teseo-LIV3F, U8 MS5637, U9 MC6470, Y1 16M, Y2 32k, Y3 32M, Y4 32k

Commit message: added attiny402 as sps
Parts:
- removed AE1: CHIP, Resistor_SMD:R_1206_3216Metric, symbol Device:Antenna
- removed C12: 100p, Capacitor_SMD:C_0402_1005Metric, symbol Device:C_Small
- removed C14, C17, C18: 1p, Capacitor_SMD:C_0402_1005Metric, symbol Device:C_Small
- removed C15: NP, Capacitor_SMD:C_0402_1005Metric, symbol Device:C_Small
- removed C16, C39, C9: 0.1u, Capacitor_SMD:C_0402_1005Metric, symbol Device:C_Small
- removed C20: 2.2p, Capacitor_SMD:C_0402_1005Metric, symbol Device:C_Small
- removed C37, C40: 10u, Capacitor_SMD:C_0402_1005Metric, symbol Device:C_Small
- removed C4: 12p, Capacitor_SMD:C_0402_1005Metric, symbol Device:C_Small
- removed C5: 10u, Capacitor_SMD:C_0805_2012Metric, symbol Device:C_Small
- removed D3: NRF_STATUS, LED_SMD:LED_0805_2012Metric, symbol Device:LED_Small_ALT
- removed D4: DC, Package_TO_SOT_SMD:SOT-23, symbol Device:D_Schottky_x2_KCom_AAK
- removed J4: DEBUG_NRF, Connector_PinHeader_1.27mm:PinHeader_2x05_P1.27mm_Vertical_SMD, symbol atlas:Conn_ARM_JTAG_SWD_10
- removed L1: 3.9n, Inductor_SMD:L_0603_1608Metric, symbol Device:L_Small
- removed L2: 15u, Inductor_SMD:L_6.3x6.3_H3, symbol Device:L_Small
- removed L4, L6: 3.9n, Inductor_SMD:L_0402_1005Metric, symbol Device:L_Small
- removed L5: NP, Inductor_SMD:L_0402_1005Metric, symbol Device:L_Small
- removed Q3: Q_NMOS_DGS, Package_TO_SOT_SMD:SOT-23, symbol Device:Q_NMOS_DGS
- removed R1, R19: 0, Resistor_SMD:R_0402_1005Metric, symbol Device:R_Small
- removed R11, R35: 1k, Resistor_SMD:R_0402_1005Metric, symbol Device:R_Small
- removed R18, R20, R21, R22, R41, R42: NP, Resistor_SMD:R_0402_1005Metric, symbol Device:R_Small
- removed R30: 10k, Resistor_SMD:R_0402_1005Metric, symbol Device:R_Small
- removed R33, R36, R39: 100k, Resistor_SMD:R_0402_1005Metric, symbol Device:R_Small
- removed SW2: Power, Button_Switch_SMD:SW_SPST_B3U-1000P, symbol Switch:SW_Push
- removed SW4: ResetNRF, Button_Switch_SMD:SW_SPST_B3U-1000P, symbol Switch:SW_Push
- removed U11: STM6601CA2BDM6F, Package_DFN_QFN:TDFN-12_2x3mm_P0.5mm, symbol Power_Management:STM6600
- removed U5: nRF52810-QCxx, Package_DFN_QFN:QFN-32-1EP_5x5mm_P0.5mm_EP3.6x3.6mm, symbol MCU_Nordic:nRF52810-QCxx
- removed Y2: 32k, Crystal:Crystal_SMD_3225-4Pin_3.2x2.5mm, symbol Device:Crystal_Small
- removed Y3: 32M, Crystal:Crystal_SMD_3225-4Pin_3.2x2.5mm, symbol Device:Crystal_Small
- added R? (x2): 100k, Resistor_SMD:R_0402_1005Metric, symbol Device:R_Small
- added U5: ATtiny402-SS, Package_SO:SOIC-8_3.9x4.9mm_P1.27mm, symbol MCU_Microchip_ATtiny:ATtiny402-SS
- C2: value 12p -> 0.1u
- SW1: value SReset -> ON_OFF
- U7: symbol atlas:Teseo-LIV3F -> atlas-rescue:Teseo-LIV3F-atlas
Connections:
- net labels added: PWR_ACK_I, PWR_CTRL_UPDI, PWR_EN_O, PWR_NR_O, PWR_SW_I, PWR_SW_O
- net labels removed: BTN_DOWN, BTN_ENTER, BTN_LEFT, BTN_RIGHT, BTN_UP, DEBUG_NRESET_NRF, DEBUG_SWDCLK_NRF, DEBUG_SWDIO_NRF, DEC1, DEC2, DEC3, DEC4, EN_MCU_PWR, EN_SD_PWR, NRF_INT, NRF_STATUS, PWR_BTN_OUT, PWR_MCU_HOLD, PWR_MCU_INT, PWR_MCU_NRST, SP4_MISO_NRF, SP4_MOSI_NRF, SP4_SCK_NRF, UART8_RX_NRF, UART8_TX_NRF, XL1_NRF, XL2_NRF
- wire segments 963 -> 817
- no-connect marks 6 -> 5
Other:
- note added: "Deep Sleep Supervisor"
- moved on the sheet: D7, J2, Q5, R25, R85, R86, R87, RN5, RN6, SW3

Commit message: rough blender model of casing further hw changes
Parts:
- removed AE2: 2088900001, atlas:2088900001, symbol Device:Antenna
- removed C2, C28, C29, C30, C45: 0.1u, Capacitor_SMD:C_0402_1005Metric, symbol Device:C_Small
- removed C43, C46: 120p, Capacitor_SMD:C_0402_1005Metric, symbol Device:C_Small
- removed F1: B39162B8813P810, Filter:Filter_1109-5_1.1x0.9mm, symbol Filter:B39162B8813P810
- removed L8: 5n6, Inductor_SMD:L_0402_1005Metric, symbol Device:L_Small
- removed Q1, Q2: Q_NMOS_DGS, Package_TO_SOT_SMD:SOT-23, symbol Device:Q_NMOS_DGS
- removed R23, R6, R7, R8, R? (x2): 100k, Resistor_SMD:R_0402_1005Metric, symbol Device:R_Small
- removed SW1: ON_OFF, Button_Switch_SMD:SW_SPST_B3U-1000P, symbol Switch:SW_Push
- removed U12: BGU7007, atlas:6-XSON_1.5x1.0mm_0.5mm, symbol atlas:BGU7007
- removed U2: W957A8MFYA5I, atlas:BGA-25_5x5_6.0x8.0mm, symbol atlas:W957D8MFYA
- removed U5: ATtiny402-SS, Package_SO:SOIC-8_3.9x4.9mm_P1.27mm, symbol MCU_Microchip_ATtiny:ATtiny402-SS
- removed U7: Teseo-LIV3F, RF_Module:ublox_MAX, symbol atlas-rescue:Teseo-LIV3F-atlas
- added C?: 0.1u, Capacitor_SMD:C_0402_1005Metric, symbol Device:C_Small
- added C?: 0.1u, Capacitor_SMD:C_0603_1608Metric, symbol Device:C_Small
- added C?: 1u, Capacitor_SMD:C_0603_1608Metric, symbol Device:C_Small
- added D?: STM_STATUS_L, LED_SMD:LED_0805_2012Metric, symbol Device:LED_Small_ALT
- added D?: STM_STATUS_0, LED_SMD:LED_0805_2012Metric, symbol Device:LED_Small_ALT
- added D?: STM_STATUS_R, LED_SMD:LED_0805_2012Metric, symbol Device:LED_Small_ALT
- added D?: MCU_3V3, LED_SMD:LED_0805_2012Metric, symbol Device:LED_Small_ALT
- added D?: GPS_3DF, LED_SMD:LED_0805_2012Metric, symbol Device:LED_Small_ALT
- added J?: DEBUG_NCP, Connector_PinHeader_1.27mm:PinHeader_2x05_P1.27mm_Vertical_SMD, symbol atlas:Conn_ARM_JTAG_SWD_10
- added J?: LPM027M128B, symbol Connector_Generic:Conn_01x10
- added J?: FLEX_12380-03, symbol Connector_Generic:Conn_01x02
- added Q?: Q_NMOS_DGS, Package_TO_SOT_SMD:SOT-23, symbol Device:Q_NMOS_DGS
- added R? (x2): 4.7k, Resistor_SMD:R_0402_1005Metric, symbol Device:R_Small
- added R? (x3): 100k, Resistor_SMD:R_0402_1005Metric, symbol Device:R_Small
- added R? (x5): 1k, Resistor_SMD:R_0402_1005Metric, symbol Device:R_Small
- added R? (x3): 10k, Resistor_SMD:R_0402_1005Metric, symbol Device:R_Small
- added R?: 100, Resistor_SMD:R_0402_1005Metric, symbol Device:R_Small
- added SW?: ResetNCP, Button_Switch_SMD:SW_SPST_B3U-1000P, symbol Switch:SW_Push
- added U?: BGM220P, symbol atlas:BGM220P
- added U?: S27KL0641DABHV023, symbol atlas:S27KL0641DABHV023
- added U?: MX25L3233FM2I-08G, Package_SO:SSOP-8_5.25x5.24mm_P1.27mm, symbol Memory_Flash:AT25SF081-XMHD-X
- D2: value STM_STATUS -> STM_STATUS_B
- R28, R29: value NP -> 4.7k
Connections:
- net labels added: DEBUG_NRESET_NCP, DEBUG_SWDCLK_NCP, DEBUG_SWDIO_NCP, DEBUG_SWO_NCP, DEBUG_SWO_STM, EXTMODE, GPS_3DF, GPS_EXTINT, GPS_FORCE_ON, I2C_SDA_SYSTEM, NCP_NRESET_STM, OCTOSPIM_P1_NCS, OPT_LCD_COM_INV, PWR_ACK_NCP, PWR_SW_IN, PWR_SW_NCP, SPI4_FLASH_CS, SPI4_FLASH_NCS, SPI4_MISO_APP, SPI4_MOSI_APP, SPI4_OPT_LCD_NCS, SPI4_SCK_APP, STM_STATUS_0, STM_STATUS_B, STM_STATUS_L, STM_STATUS_R, SW_C, SW_L, SW_R, T3C1_LCD_BL, USART3_CTS_NCP, USART3_RTS_NCP, USART3_RX_NCP, USART3_TX_NCP
- net labels removed: GPS_ANT_OFF, GPS_RESET, GPS_VCC_RF, GPS_WAKEUP, LTDC_G3, MCU_LV_RESET, OCTOSPIM_P1_NPLK, PWR_CTRL_UPDI, PWR_NR_O, PWR_SW_I, PWR_SW_O, STM_STATUS, TIM4_CH3_LCD_BL_PWM
- wire segments 817 -> 863
- no-connect marks 5 -> 6
Other:
- note added: "On button hold, if shutdown DSS holds PWR_EN, starts timeout for PWR_ACK. If timeout is not met, cycle power (max 3 times).\n\nIf PWR_ACK is successful, then the device remains powered up. If button is short pressed, no action is taken by DSS and the signal is passed to PWR_SW_O. If the button is long pressed, the signal is also sent to PWR_SW_O, but PWR_ACK is expected. Once PWR_ACK is released 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"
- note removed: "Deep Sleep Supervisor"
- moved on the sheet: C1, C11, C19, C21, C22, C23, C24, C25, C26, C3, C32, C33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

Commit message: begining hw layout
Parts:
- added AE1: Antenna_Shield, Connector_Coaxial:U.FL_Hirose_U.FL-R-SMT-1_Vertical, symbol Device:Antenna_Shield
- added C4: 56p, Capacitor_SMD:C_0402_1005Metric, symbol Device:C_Small
- added F1: SF14-1575F5UUC1, Filter:Filter_1411-5_1.4x1.1mm, symbol Filter:SF14-1575F5UUC1
- added R21, R22, R23, R30, R39: 0, Resistor_SMD:R_0402_1005Metric, symbol Device:R_Small
- added R45, R48: 100, Resistor_SMD:R_0402_1005Metric, symbol Device:R_Small
- added U11: L96-M33, atlas:L96, symbol atlas:L96-M33
- added U12: BGU7007, atlas:6-XSON_1.5x1.0mm_0.5mm, symbol atlas:BGU7007
- J6: renamed from J?; footprint (none) -> Connector_FFC-FPC:Hirose_FH12-10S-0.5SH_1x10-1MP_P0.50mm_Horizontal
- J7: renamed from J?; footprint (none) -> Connector_FFC-FPC:TE_84952-4_1x04-1MP_P1.0mm_Horizontal
- J8: footprint Connector_Card:microSD_HC_Hirose_DM3D-SF -> Connector_Card:microSD_HC_Hirose_DM3AT-SF-PEJM5
- L10, L3, L7, L9: footprint Inductor_SMD:L_6.3x6.3_H3 -> Inductor_SMD:L_Bourns-SRN4018
- U2: renamed from U?; footprint (none) -> atlas:BGA-25_5x5_6.0x8.0mm
- U7: renamed from U?; footprint (none) -> atlas:BGM220P
- gave numbers to parts that had none: 26
Connections:
- net DEBUG_NRESET_STM: now also R22.2
- net GND: now also AE1.2 (Shield), F1.2, F1.3, F1.5, U11.10 (GND), U11.11 (GND), U11.12 (GND), U11.13 (GND), U11.14 (GND), U11.15 (GND), U11.18 (GND), U11.19 (GND), U11.21 (GND), U11.22 (GND), U11.27 (GND), U11.31 (GND), U11.4 (GND), U11.5 (GND), U12.1 (G), U12.2 (G)
- net GPS_1PPS: now also U11.29 (PPS)
- net GPS_3DF: now also U11.2 (3D_FIX)
- net I2C1_SCL_SYSTEM: no longer U1.59 (PD12)
- net I2C1_SDA_SYSTEM: no longer U1.60 (PD13)
- net I2C_SCL_SENSOR: now also R23.2
- net I2C_SDA_SENSOR: now also R30.2
- net LPUART1_RX_GPS: now also U11.25 (TXD1)
- net LPUART1_TX_GPS: now also U11.26 (RXD1)
- net VCC_BACKUP: now also U11.8 (V_BCKP)
- net VCC_MCU_3V3: now also R21.2, R48.1, U11.9 (VCC)
- new net: R39.2, U11.16 (RF_OUT)
- new net: C4.2, R39.1, U11.17 (RF_IN)
- new net: R21.1, R22.1, U11.23 (~RESET)
- new net: R30.1, U11.3 (I2C_SDA)
- new net: R45.2, U11.30 (ANTON)
- new net: R23.1, U11.6 (I2C_SCL)
- new net: F1.4, U12.3
- new net: R48.2, U12.4 (VCC)
- new net: R45.1, U12.5
- new net: C4.1, U12.6
- new net: AE1.1 (A), F1.1
- new net I2C4_SCL_SYSTEM: U1.59 (PD12)
- new net I2C4_SDA_SYSTEM: U1.60 (PD13)
- no-connect marks 6 -> 8
Other:
- note removed: "On button hold, if shutdown DSS holds PWR_EN, starts timeout for PWR_ACK. If timeout is not met, cycle power (max 3 times).\n\nIf PWR_ACK is successful, then the device remains powered up. If button is short pressed, no action is taken by DSS and the signal is passed to PWR_SW_O. If the button is long pressed, the signal is also sent to PWR_SW_O, but PWR_ACK is expected. Once PWR_ACK is released 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"
- moved on the sheet: C2, C32, C33, C34, C56, C57, C58, C59, C60, C61, C62, C63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

Commit message: layout of sd, octo, place sensors, connectors
Parts:
- removed RN5, RN6: R_Pack04, Resistor_SMD:R_Array_Concave_4x0402, symbol Device:R_Pack04
- J8: footprint Connector_Card:microSD_HC_Hirose_DM3AT-SF-PEJM5 -> Connector_Card:microSD_HC_Hirose_DM3BT-DSF-PEJS
- SW1, SW3: footprint Button_Switch_SMD:SW_SPST_B3U-1000P -> Jumper:SolderJumper-2_P1.3mm_Open_Pad1.0x1.5mm
Connections:
- net OCTOSPIM_P1_NPS is gone; now on net OCTOSPIM_P1_NCS: U2.A3 (CS#)
- net GPS_EXTINT: now also U11.7 (EXTINT0)
- net GPS_FORCE_ON: now also U11.28 (FORCE_ON)
- net I2C4_SCL_SYSTEM: now also R23.2, U10.5 (SCL), U6.8 (SCL)
- net I2C4_SDA_SYSTEM: now also R30.2, R33.2, R35.2, U10.6 (SDA), U6.7 (SDA)
- net LTDC_B4: now also RN3.4 (R4.1); no longer RN3.1 (R1.1)
- net LTDC_B5: now also RN3.3 (R3.1); no longer RN3.2 (R2.1)
- net LTDC_B6: now also RN3.2 (R2.1); no longer RN3.3 (R3.1)
- net LTDC_B7: now also RN3.1 (R1.1); no longer RN3.4 (R4.1)
- net LTDC_CK: now also RN4.4 (R4.1); no longer RN4.1 (R1.1)
- net LTDC_DE: now also RN4.3 (R3.1); no longer RN4.2 (R2.1)
- net LTDC_G4: now also RN2.4 (R4.1); no longer RN2.1 (R1.1)
- net LTDC_G5: now also RN2.3 (R3.1); no longer RN2.2 (R2.1)
- net LTDC_G6: now also RN2.2 (R2.1); no longer RN2.3 (R3.1)
- net LTDC_G7: now also RN2.1 (R1.1); no longer RN2.4 (R4.1)
- net LTDC_HS: now also RN4.2 (R2.1); no longer RN4.3 (R3.1)
- net LTDC_R4: now also RN1.4 (R4.1); no longer RN1.1 (R1.1)
- net LTDC_R5: now also RN1.3 (R3.1); no longer RN1.2 (R2.1)
- net LTDC_R6: now also RN1.2 (R2.1); no longer RN1.3 (R3.1)
- net LTDC_R7: now also RN1.1 (R1.1); no longer RN1.4 (R4.1)
- net LTDC_VS: now also RN4.1 (R1.1); no longer RN4.4 (R4.1)
- net SDMMC1_CK: now also U13.4 (A1); no longer U13.8 (A5)
- net SDMMC1_CKIN: now also U13.5 (A2); no longer U13.7 (A4)
- net SDMMC1_CMD: now also U13.3 (A0); no longer U13.6 (A3)
- net SDMMC1_D0: now also U13.8 (A5); no longer U13.9 (A6)
- net SDMMC1_D1: now also U13.9 (A6); no longer U13.10 (A7)
- net SDMMC1_D2: now also U13.7 (A4); no longer U13.4 (A1)
- net SDMMC1_D3: now also U13.6 (A3); no longer U13.5 (A2)
- net SD_CLK: now also U13.16 (B2), U13.17 (B1); no longer U13.13 (B5), U13.14 (B4)
- net SD_CMD: now also U13.18 (B0); no longer U13.15 (B3)
- net SD_D0: now also U13.13 (B5); no longer U13.12 (B6)
- net SD_D1: now also U13.12 (B6); no longer U13.11 (B7)
- net SD_D2: now also U13.14 (B4); no longer U13.17 (B1)
- net SD_D3: now also U13.15 (B3); no longer U13.16 (B2)
- net at R89.1: now also U13.11 (B7); no longer U13.18 (B0)
- net at R88.1: now also U13.10 (A7); no longer U13.3 (A0)
- net I2C1_SCL_SYSTEM renamed I2C1_SCL_SENSOR
- net I2C1_SCL_SENSOR: now also R28.2, U8.3 (SCL), U9.12 (SCL); no longer U10.5 (SCL), U6.8 (SCL)
- removed net I2C1_SDA_SYSTEM: J3.2 (Pin_2), R33.2, R35.2, U1.93 (PB7), U10.6 (SDA), U6.7 (SDA)
- removed net I2C_SCL_SENSOR: R23.2, R28.2, U8.3 (SCL), U9.12 (SCL)
- net I2C_SDA_SENSOR renamed I2C1_SDA_SENSOR
- net I2C1_SDA_SENSOR: now also J3.2 (Pin_2), U1.93 (PB7); no longer R30.2
Other:
- note removed: "Place under U13"
- moved on the sheet: AE1, C32, C33, C34, C38, C4, C59, C60, F1, J3, R21, R22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

Commit message: removed bgm220, compacted layout, mounting holes, dss, power supply
Parts:
- removed AE1: Antenna_Shield, Connector_Coaxial:U.FL_Hirose_U.FL-R-SMT-1_Vertical, symbol Device:Antenna_Shield
- removed C36, C42: 10u, Capacitor_SMD:C_0805_2012Metric, symbol Device:C_Small
- removed F1: SF14-1575F5UUC1, Filter:Filter_1411-5_1.4x1.1mm, symbol Filter:SF14-1575F5UUC1
- removed J4: DEBUG_NCP, Connector_PinHeader_1.27mm:PinHeader_2x05_P1.27mm_Vertical_SMD, symbol atlas:Conn_ARM_JTAG_SWD_10
- removed R45, R48: 100, Resistor_SMD:R_0402_1005Metric, symbol Device:R_Small
- removed R74, R77: NP, Resistor_SMD:R_0402_1005Metric, symbol Device:R_Small
- removed R88, R89: 0, Resistor_SMD:R_0402_1005Metric, symbol Device:R_Small
- removed SW1: ResetNCP, Jumper:SolderJumper-2_P1.3mm_Open_Pad1.0x1.5mm, symbol Switch:SW_Push
- removed U12: BGU7007, atlas:6-XSON_1.5x1.0mm_0.5mm, symbol atlas:BGU7007
- removed U7: BGM220P, atlas:BGM220P, symbol atlas:BGM220P
- added C12, C14, C15, C16: 4.7u, Capacitor_SMD:C_0603_1608Metric, symbol Device:C_Small
- added J11: UART3_EXT, Connector_PinHeader_1.00mm:PinHeader_1x06_P1.00mm_Vertical, symbol Connector_Generic:Conn_01x06
- added J4: UPDI_DSS, Connector_PinHeader_1.00mm:PinHeader_1x03_P1.00mm_Vertical, symbol Connector_Generic:Conn_01x03
- added Q2: Q_NMOS_DGS, Package_TO_SOT_SMD:SOT-23, symbol Device:Q_NMOS_DGS
- added U7: ATtiny402-SS, Package_SO:SOIC-8_3.9x4.9mm_P1.27mm, symbol MCU_Microchip_ATtiny:ATtiny402-SS
- C35: value 0.1u -> 1u; footprint Capacitor_SMD:C_0402_1005Metric -> Capacitor_SMD:C_0603_1608Metric
- C4: value 56p -> 4.7u; footprint Capacitor_SMD:C_0402_1005Metric -> Capacitor_SMD:C_0603_1608Metric
- C44: value 10u -> 4.7u; footprint Capacitor_SMD:C_0805_2012Metric -> Capacitor_SMD:C_0603_1608Metric
- J5: footprint Connector_JST:JST_GH_SM03B-GHS-TB_1x03-1MP_P1.25mm_Horizontal -> Connector_PinHeader_1.00mm:PinHeader_1x03_P1.00mm_Vertical
- L10, L9: footprint Inductor_SMD:L_Bourns-SRN4018 -> Inductor_SMD:L_Taiyo-Yuden_MD-3030
- R20: value 10k -> 10; footprint Resistor_SMD:R_0402_1005Metric -> Resistor_SMD:R_0815_2038Metric
- R40: footprint Resistor_SMD:R_0402_1005Metric -> Resistor_SMD:R_0815_2038Metric
- R43: value 0 -> 100k
- R44: value 0 -> 10k
- Y4: footprint Crystal:Crystal_SMD_3225-4Pin_3.2x2.5mm -> Crystal:Crystal_SMD_3215-2Pin_3.2x1.5mm
Connections:
- net DEBUG_NRESET_NCP is gone; now on net GND: R20.1
- net PWR_ACK_I is gone; now on net PWR_EN_O: R6.1
- net VDD_SD_1V8 is gone; now on net VDD_SD_IO_3V3_1V8: C63.1, U14.5 (OUT)
- net BQ25611_INT: now also U1.58 (PD11); no longer U1.97 (PE0)
- net CELL_POS: now also C14.2
- net EN_LCD_PWR: now also R47.2, U16.3 (EN)
- net GND: now also C4.1, J10.1 (Pin_1), J10.2 (Pin_2), J10.29 (Pin_29), U13.10 (A7), U13.11 (B7), C12.1, C14.1, C15.1, C16.1, J11.1 (Pin_1), J4.1 (Pin_1), Q2.3 (S), U7.8 (GND); no longer J10.12 (Pin_12), J10.39 (Pin_39), J10.40 (Pin_40)
- net LC709203_INT: now also U1.57 (PD10); no longer U1.85 (PD4)
- net LTDC_B4: now also J10.21 (Pin_21), J10.25 (Pin_25), RN3.1 (R1.1); no longer J10.16 (Pin_16), J10.20 (Pin_20), RN3.4 (R4.1)
- net LTDC_B5: now also J10.22 (Pin_22), J10.26 (Pin_26), RN3.2 (R2.1); no longer J10.15 (Pin_15), J10.19 (Pin_19), RN3.3 (R3.1)
- net LTDC_B6: now also J10.23 (Pin_23), J10.27 (Pin_27), RN3.3 (R3.1); no longer J10.14 (Pin_14), J10.18 (Pin_18), RN3.2 (R2.1)
- net LTDC_B7: now also J10.24 (Pin_24), J10.28 (Pin_28), RN3.4 (R4.1); no longer J10.13 (Pin_13), J10.17 (Pin_17), RN3.1 (R1.1)
- net LTDC_CK: now also J10.30 (Pin_30), RN4.1 (R1.1); no longer J10.11 (Pin_11), RN4.4 (R4.1)
- net LTDC_DE: now also J10.31 (Pin_31), RN4.2 (R2.1); no longer J10.10 (Pin_10), RN4.3 (R3.1)
- net LTDC_G4: now also J10.13 (Pin_13), J10.17 (Pin_17), RN2.1 (R1.1); no longer J10.24 (Pin_24), J10.28 (Pin_28), RN2.4 (R4.1)
- net LTDC_G5: now also J10.14 (Pin_14), J10.18 (Pin_18), RN2.2 (R2.1); no longer J10.23 (Pin_23), J10.27 (Pin_27), RN2.3 (R3.1)
- net LTDC_G6: now also J10.15 (Pin_15), J10.19 (Pin_19), RN2.3 (R3.1); no longer J10.22 (Pin_22), J10.26 (Pin_26), RN2.2 (R2.1)
- net LTDC_G7: now also J10.16 (Pin_16), J10.20 (Pin_20), RN2.4 (R4.1); no longer J10.21 (Pin_21), J10.25 (Pin_25), RN2.1 (R1.1)
- net LTDC_HS: now also J10.32 (Pin_32), RN4.3 (R3.1); no longer J10.9 (Pin_9), RN4.2 (R2.1)
- net LTDC_R4: now also J10.5 (Pin_5), J10.9 (Pin_9), RN1.1 (R1.1); no longer J10.32 (Pin_32), J10.36 (Pin_36), RN1.4 (R4.1)
- net LTDC_R5: now also J10.10 (Pin_10), J10.6 (Pin_6), RN1.2 (R2.1); no longer J10.31 (Pin_31), J10.35 (Pin_35), RN1.3 (R3.1)
- net LTDC_R6: now also J10.11 (Pin_11), J10.7 (Pin_7), RN1.3 (R3.1); no longer J10.30 (Pin_30), J10.34 (Pin_34), RN1.2 (R2.1)
- net LTDC_R7: now also J10.12 (Pin_12), J10.8 (Pin_8), RN1.4 (R4.1); no longer J10.29 (Pin_29), J10.33 (Pin_33), RN1.1 (R1.1)
- net LTDC_VS: now also J10.33 (Pin_33), RN4.4 (R4.1); no longer J10.8 (Pin_8), RN4.1 (R1.1)
- net MC6470_INTA: now also U1.88 (PD7); no longer U1.57 (PD10)
- net MC6470_INTM: now also U1.87 (PD6); no longer U1.58 (PD11)
- net PWR_EN_O: now also R44.2, U7.2 (PA6); no longer R1.2
- net PWR_SW_IN: now also U7.4 (PA1)
- net SDMMC1_CK: now also U13.6 (A3); no longer U13.4 (A1)
- net SDMMC1_CMD: now also U13.7 (A4); no longer U13.3 (A0)
- net SDMMC1_D0: now also U13.4 (A1); no longer U13.8 (A5)
- net SDMMC1_D1: now also U13.3 (A0); no longer U13.9 (A6)
- net SDMMC1_D2: now also U13.9 (A6); no longer U13.7 (A4)
- net SDMMC1_D3: now also U13.8 (A5); no longer U13.6 (A3)
- net SD_CLK: now also U13.15 (B3); no longer U13.17 (B1)
- net SD_CMD: now also U13.14 (B4); no longer U13.18 (B0)
- net SD_D0: now also U13.17 (B1); no longer U13.13 (B5)
- net SD_D1: now also U13.18 (B0); no longer U13.12 (B6)
- net SD_D2: now also U13.12 (B6); no longer U13.14 (B4)
- net SD_D3: now also U13.13 (B5); no longer U13.15 (B3)
- net T3C1_LCD_BL: now also Q2.2 (G); no longer R47.2, U16.3 (EN)
- net USART3_CTS_NCP: now also J11.5 (Pin_5)
- net USART3_RTS_NCP: now also J11.6 (Pin_6)
- net USART3_RX_NCP: now also J11.3 (Pin_3)
- net USART3_TX_NCP: now also J11.4 (Pin_4)
- net VCC_BACKUP: now also R44.1, J4.2 (Pin_2), U7.1 (VCC)
- net VCC_MCU_3V3: now also C62.1, U14.1 (IN), U14.3 (EN), J11.2 (Pin_2); no longer R20.2, R43.1, R44.1
- net VCC_SYS: now also C16.2
- net VDD_SD_IO_3V3_1V8: now also R43.1, R75.2; no longer U13.20 (~OE)
- net ~USB_DET: now also U7.5 (PA2)
- net at R31.1, U10.22 (REGN): now also C15.2
- net at U10.23 (PMID): now also C4.2, C12.2
- net at R39.1, U11.17 (RF_IN): no longer C4.2
- net at R84.2: now also J10.40 (Pin_40); no longer J10.1 (Pin_1)
- net at R83.2: now also J10.39 (Pin_39); no longer J10.2 (Pin_2)
- net at J10.3 (Pin_3): now also C54.1, C55.1, J10.4 (Pin_4), R81.1; no longer R82.2
- net at C51.1, C53.1, R80.1: now also J10.35 (Pin_35), J10.36 (Pin_36); no longer J10.6 (Pin_6)
- net at R43.2: now also U13.20 (~OE); no longer U14.3 (EN)
- net at C49.2, U16.4 (COMP): now also Q2.1 (D)
- net at J9.4 (Pin_4), U16.6 (FB): now also R20.2
- net PWR_ACK_NCP renamed PWR_ACK_DSS
- net PWR_ACK_DSS: now also R1.2, U7.7 (PA3)
- net PWR_SW_NCP renamed PWR_SW_DSS
- net PWR_SW_DSS: now also U7.3 (PA7)
- new net: J10.38 (Pin_38), R82.2
- new net UDPI_DSS: J4.3 (Pin_3), U7.6 (~RESET~/PA0)
- now unconnected: J10.37 (Pin_37)
Other:
- moved on the sheet: C48, C59, C60, R46, R47, R6
