File: atlas_hw/atlas.sch (KiCad schematic (older format))
At the start: 163 parts, among them J1 USB_C_Receptacle_USB2.0, J10 PSP_LCD, J11 UART3_EXT, J2 DEBUG_STM, J3 PSP_TOUCH, J4 UPDI_DSS, J5 CELL_THERM, J6 LPM027M128B, J7 FLEX_12380-03, J8 Micro_SD_Card_Det, J9 PSP_LCD_BL, Q1 Q_NMOS_DGS, Q2 Q_NMOS_DGS, Q4 Q_NMOS_DGS, Q5 Q_NMOS_DGS, SW3 ResetSTM, U1 STM32H723VITx, U10 BQ25611D, U11 L96-M33, U13 LSF0108, U14 NPP600SNADJ, U15 TPS61073, U16 PAM2841, U2 S27KL0641DABHV023, U3 MCP1811B, U4 TLV62569DBV, U5 MX25L3233FM2I-08G, U6 LC709203F, U7 ATtiny402-SS, U8 MS5637, U9 MC6470, Y1 16M, Y4 32k

Commit message: further layout shrink, button board
Parts:
- added C17, C18: 0.1u, Capacitor_SMD:C_0402_1005Metric, symbol Device:C_Small
- added J12: IO_EXT, Connector_FFC-FPC:Hirose_FH12-10S-0.5SH_1x10-1MP_P0.50mm_Horizontal, symbol Connector_Generic:Conn_01x10
- added J13: IO_MAIN, Connector_FFC-FPC:Hirose_FH12-10S-0.5SH_1x10-1MP_P0.50mm_Horizontal, symbol Connector_Generic:Conn_01x10
- added R45, R48, R50: 100k, Resistor_SMD:R_0805_2012Metric, symbol Device:R_Small
- added SW1: BTN_L_EXT, Button_Switch_SMD:SW_SPST_B3S-1000, symbol Switch:SW_Push
- added SW2: BTN_0_EXT, Button_Switch_SMD:SW_SPST_B3S-1000, symbol Switch:SW_Push
- added SW4: BTN_R_EXT, Button_Switch_SMD:SW_SPST_B3S-1000, symbol Switch:SW_Push
- added SW5: BTN_PWR_EXT, Button_Switch_SMD:SW_SPST_B3U-1000P, symbol Switch:SW_Push
- C13, C7: value 1u -> 10u; footprint Capacitor_SMD:C_0603_1608Metric -> Capacitor_SMD:C_0805_2012Metric
- D6: footprint Diode_SMD:D_SOD-123F -> Diode_SMD:D_SOD-110
- J7: footprint Connector_FFC-FPC:TE_84952-4_1x04-1MP_P1.0mm_Horizontal -> Connector_PinHeader_1.00mm:PinHeader_1x02_P1.00mm_Vertical
- R11, R18, R19: footprint Resistor_SMD:R_0402_1005Metric -> Resistor_SMD:R_0805_2012Metric
- R20: footprint Resistor_SMD:R_0815_2038Metric -> Resistor_SMD:R_0603_1608Metric
- R40: value 0 -> 100k; footprint Resistor_SMD:R_0815_2038Metric -> Resistor_SMD:R_0805_2012Metric
- R46: footprint Resistor_SMD:R_0402_1005Metric -> Resistor_SMD:R_0612_1632Metric
Connections:
- net GND: now also D10.1 (K), D8.1 (K), D9.1 (K), J5.3 (Pin_3), U13.18 (B0), U13.19 (VCCB), U13.3 (A0), C17.1, C18.2, J12.1 (Pin_1), J12.10 (Pin_10), J13.1 (Pin_1), J13.10 (Pin_10), SW1.2, SW2.2, SW4.2, SW5.2; no longer R11.2, R18.2, R19.2, R40.1, U13.1 (GND), U13.10 (A7), U13.11 (B7), U13.21 (NC)
- net SDMMC1_CK: now also U13.7 (A4); no longer U13.6 (A3)
- net SDMMC1_CKIN: now also U13.8 (A5); no longer U13.5 (A2)
- net SDMMC1_CMD: now also U13.6 (A3); no longer U13.7 (A4)
- net SDMMC1_D0: now also U13.9 (A6); no longer U13.4 (A1)
- net SDMMC1_D1: now also U13.10 (A7); no longer U13.3 (A0)
- net SDMMC1_D2: now also U13.4 (A1); no longer U13.9 (A6)
- net SDMMC1_D3: now also U13.5 (A2); no longer U13.8 (A5)
- net SD_CLK: now also U13.13 (B5), U13.14 (B4); no longer U13.15 (B3), U13.16 (B2)
- net SD_CMD: now also U13.15 (B3); no longer U13.14 (B4)
- net SD_D0: now also U13.12 (B6); no longer U13.17 (B1)
- net SD_D1: now also U13.11 (B7); no longer U13.18 (B0)
- net SD_D2: now also U13.17 (B1); no longer U13.12 (B6)
- net SD_D3: now also U13.16 (B2); no longer U13.13 (B5)
- net STM_STATUS_0: now also J13.5 (Pin_5); no longer D9.2 (A)
- net STM_STATUS_B: now also U1.97 (PE0)
- net STM_STATUS_L: now also J13.3 (Pin_3); no longer D8.2 (A)
- net STM_STATUS_R: now also J13.7 (Pin_7); no longer D10.2 (A)
- net SW_L: now also J13.2 (Pin_2)
- net SW_R: now also J13.6 (Pin_6)
- net VCC_MCU_3V3: now also U13.20 (~OE), C18.1, J13.9 (Pin_9); no longer U13.2 (VCCA)
- net VDD_SD_IO_3V3_1V8: now also U13.1 (GND), U13.21 (NC); no longer U13.19 (VCCB)
- net at R43.2: now also U13.2 (VCCA); no longer U13.20 (~OE)
- net STM_STATUS_L_EXT: now reaches R11.1
- net STM_STATUS_L_EXT: now also J12.9 (Pin_9); no longer D8.1 (K)
- net STM_STATUS_0_EXT: now reaches R18.1
- net STM_STATUS_0_EXT: now also J12.8 (Pin_8); no longer D9.1 (K)
- net STM_STATUS_R_EXT: now reaches R19.1
- net STM_STATUS_R_EXT: now also J12.7 (Pin_7); no longer D10.1 (K)
- net CELL_NEG renamed SW_L_EXT
- net SW_L_EXT: now also J12.3 (Pin_3), SW1.1; no longer J5.3 (Pin_3)
- net PWR_SW_IN renamed SW_PWR
- net SW_PWR: now also J13.8 (Pin_8)
- new net: D8.2 (A), R11.2
- new net: D9.2 (A), R18.2
- new net: D10.2 (A), R19.2
- new net SW_0: J13.4 (Pin_4)
- new net SW_0_EXT: J12.4 (Pin_4), R45.2, SW2.1
- new net SW_PWR_EXT: J12.6 (Pin_6), R50.2, SW5.1
- new net SW_R_EXT: J12.5 (Pin_5), R48.2, SW4.1
- new net VCC_3V3_EXT: C17.2, J12.2 (Pin_2), R40.1, R45.1, R48.1, R50.1
Other:
- moved on the sheet: D1, D10, D2, D3, D4, D7, D8, D9, J11, Q5, R10, R11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

Commit message: passive placement
Parts:
- removed C55: 0.1u, Capacitor_SMD:C_0402_1005Metric, symbol Device:C_Small
- removed R2, R80, R81: 0, Resistor_SMD:R_0402_1005Metric, symbol Device:R_Small
- removed R46: 0, Resistor_SMD:R_0612_1632Metric, symbol Device:R_Small
- added C20: 1u, Capacitor_SMD:C_0603_1608Metric, symbol Device:C_Small
- added C28: 0.1u, Capacitor_SMD:C_0402_1005Metric, symbol Device:C_Small
- J11: footprint Connector_PinHeader_1.00mm:PinHeader_1x06_P1.00mm_Vertical -> Connector_PinHeader_1.00mm:PinHeader_1x06_P1.00mm_Vertical_SMD_Pin1Left
- R1, R25, R44, R6: value 10k -> 100k
Connections:
- net GND: now also U1.19 (VSSA), U13.1 (GND), U13.10 (A7), U13.11 (B7), U13.21 (NC), C20.2, C28.1; no longer U13.18 (B0), U13.19 (VCCB), U13.3 (A0)
- net RCC_OSC_IN: now also Y1.2; no longer Y1.1
- net RCC_OSC_OUT: now also Y1.1; no longer Y1.2
- net SDMMC1_CK: now also U13.6 (A3); no longer U13.7 (A4)
- net SDMMC1_CKIN: now also U13.5 (A2); no longer U13.8 (A5)
- net SDMMC1_CMD: now also U13.7 (A4); no longer U13.6 (A3)
- net SDMMC1_D0: now also U13.4 (A1); no longer U13.9 (A6)
- net SDMMC1_D1: now also U13.3 (A0); no longer U13.10 (A7)
- net SDMMC1_D2: now also U13.9 (A6); no longer U13.4 (A1)
- net SDMMC1_D3: now also U13.8 (A5); no longer U13.5 (A2)
- net SD_CLK: now also U13.15 (B3), U13.16 (B2); no longer U13.13 (B5), U13.14 (B4)
- net SD_CMD: now also U13.14 (B4); no longer U13.15 (B3)
- net SD_D0: now also U13.17 (B1); no longer U13.12 (B6)
- net SD_D1: now also U13.18 (B0); no longer U13.11 (B7)
- net SD_D2: now also U13.12 (B6); no longer U13.17 (B1)
- net SD_D3: now also U13.13 (B5); no longer U13.16 (B2)
- net USART3_CTS_NCP: now also J11.3 (Pin_3); no longer J11.5 (Pin_5)
- net USART3_RTS_NCP: now also J11.4 (Pin_4); no longer J11.6 (Pin_6)
- net USART3_RX_NCP: now also J11.6 (Pin_6); no longer J11.3 (Pin_3)
- net USART3_TX_NCP: now also J11.5 (Pin_5); no longer J11.4 (Pin_4)
- net VCC_BACKUP: now also C28.2; no longer R1.1
- net VCC_LCD_PWR: now also C51.1, C53.1, J10.35 (Pin_35), J10.36 (Pin_36)
- net VCC_MCU_3V3: now also C54.1, J10.3 (Pin_3), J10.4 (Pin_4), R1.1, U13.2 (VCCA), C20.1; no longer U13.20 (~OE)
- net VCC_SYS: now also C48.2, L10.1, U16.2 (VIN)
- net VDD_SD_IO_3V3_1V8: now also U13.19 (VCCB); no longer U13.1 (GND), U13.21 (NC)
- net at R43.2: now also U13.20 (~OE); no longer U13.2 (VCCA)
Other:
- moved on the sheet: R1
Changed lines of the file:
@@
 	3750 4000 3750 4350
 $Comp
-L Device:R_Small R2
-U 1 1 689C7FDD
-P 3450 10000
-F 0 "R2" V 3550 10100 50  0000 C CNN
-F 1 "0" V 3550 9900 50  0000 C CNN
-F 2 "Resistor_SMD:R_0402_1005Metric" H 3450 10000 50  0001 C CNN
-F 3 "~" H 3450 10000 50  0001 C CNN
-	1    3450 10000
-	0    1    1    0
-$EndComp
-Wire Wire Line
-	3550 10000 3650 10000
-Wire Wire Line
-	3650 10000 3650 9850
-Wire Wire Line
-	3150 9900 3150 10000
-Connection ~ 3150 10000
-Wire Wire Line
-	3150 10000 3150 10100
-$Comp
 L power:GND #PWR09
 U 1 1 68B4FC01
@@
 	1    0    0    -1
 $EndComp
-Wire Wire Line
-	3150 10000 3350 10000
 Text Label 1700 9550 0    39   ~ 0
 GPS_EXTINT
@@
 F 3 "~" H 1300 6550 50  0001 C CNN
 	1    1300 6550
-	1    0    0    -1
+	-1   0    0    1
 $EndComp
 Wire Wire Line
@@
 Wire Wire Line
 	20050 3850 19950 3850
-$Comp
-L Device:C_Small C55
-U 1 1 7BDF01FE
-P 19950 4050
-F 0 "C55" H 19858 4096 50  0000 R CNN
-F 1 "0.1u" H 19858 4005 50  0000 R CNN
-F 2 "Capacitor_SMD:C_0402_1005Metric" H 19950 4050 50  0001 C CNN
-F 3 "~" H 19950 4050 50  0001 C CNN
-	1    19950 4050
-	1    0    0    -1
-$EndComp
 Wire Wire Line
 	19950 3950 19950 3850
@@
 Text Label 18400 7450 2    39   ~ 0
 LTDC_DE
-$Comp
-L Device:R_Small R81
-U 1 1 805CA4FA
-P 19450 3850
-F 0 "R81" V 19250 3850 50  0000 C CNN
-F 1 "0" V 19350 3850 50  0000 C CNN
-F 2 "Resistor_SMD:R_0402_1005Metric" H 19450 3850 50  0001 C CNN
-F 3 "~" H 19450 3850 50  0001 C CNN
-	1    19450 3850
-	0    1    1    0
-$EndComp
-Wire Wire Line
-	19550 3850 19600 3850
 Connection ~ 19600 3850
-Wire Wire Line
-	19350 3850 18900 3850
-$Comp
-L Device:R_Small R80
-U 1 1 80793387
-P 19300 7050
-F 0 "R80" V 19100 7050 50  0000 C CNN
-F 1 "0" V 19200 7050 50  0000 C CNN
-F 2 "Resistor_SMD:R_0402_1005Metric" H 19300 7050 50  0001 C CNN
-F 3 "~" H 19300 7050 50  0001 C CNN
-	1    19300 7050
-	0    1    1    0
-$EndComp
-Wire Wire Line
-	19450 7050 19400 7050
 Connection ~ 19450 7050
-Wire Wire Line
-	19200 7050 18800 7050
-$Comp
-L Device:R_Small R46
-U 1 1 80A4DDE0
-P 16500 2400
-F 0 "R46" V 16300 2400 50  0000 C CNN
-F 1 "0" V 16400 2400 50  0000 C CNN
-F 2 "Resistor_SMD:R_0612_1632Metric" H 16500 2400 50  0001 C CNN
-F 3 "~" H 16500 2400 50  0001 C CNN
-	1    16500 2400
-	0    1    1    0
-$EndComp
-Wire Wire Line
-	16600 2400 16950 2400
 Connection ~ 16950 2400
-Wire Wire Line
-	16400 2400 15800 2400
 Connection ~ 19300 2400
 Wire Wire Line
@@
 P 7400 14150
 F 0 "R25" V 7500 14050 50  0000 C CNN
-F 1 "10k" V 7500 14250 50  0000 C CNN
+F 1 "100k" V 7500 14250 50  0000 C CNN
 F 2 "Resistor_SMD:R_0402_1005Metric" H 7400 14150 50  0001 C CNN
 F 3 "~" H 7400 14150 50  0001 C CNN
@@
 	4350 4650 5200 4650
 Wire Wire Line
-	4350 7550 5200 7550
-Wire Wire Line
 	4350 4950 5200 4950
 Text Label 5200 4650 2    39   ~ 0
@@
 	1    0    0    -1
 $EndComp
-Text Label 6800 11500 0    39   ~ 8
+Text Label 6350 11500 0    39   ~ 8
 VCC_BACKUP
 Wire Wire Line
@@
 P 8550 12650
 F 0 "R6" H 8700 12600 50  0000 C CNN
-F 1 "10k" H 8700 12700 50  0000 C CNN
+F 1 "100k" H 8700 12700 50  0000 C CNN
 F 2 "Resistor_SMD:R_0402_1005Metric" H 8550 12650 50  0001 C CNN
 F 3 "~" H 8550 12650 50  0001 C CNN
@@
 Wire Wire Line
 	9100 12400 8100 12400
-Wire Wire Line
-	9100 12200 8250 12200
 $Comp
 L power:GND #PWR0125
@@
 	1    0    0    -1
 $EndComp
-Text Label 10950 7650 2    39   ~ 0
-USART3_RX_NCP
-Text Label 10950 7750 2    39   ~ 0
-USART3_TX_NCP
-Text Label 10950 7850 2    39   ~ 0
-USART3_CTS_NCP
-Text Label 10950 7950 2    39   ~ 0
-USART3_RTS_NCP
-Wire Wire Line
-	10400 7950 10950 7950
-Wire Wire Line
-	10400 7850 10950 7850
-Wire Wire Line
-	10400 7750 10950 7750
 Wire Wire Line
 	10400 7650 10950 7650
@@
 P 8550 11650
 F 0 "R44" H 8700 11600 50  0000 C CNN
-F 1 "10k" H 8700 11700 50  0000 C CNN
+F 1 "100k" H 8700 11700 50  0000 C CNN
 F 2 "Resistor_SMD:R_0402_1005Metric" H 8550 11650 50  0001 C CNN
 F 3 "~" H 8550 11650 50  0001 C CNN
@@
 L Device:R_Small R1
 U 1 1 61100176
-P 8250 11650
-F 0 "R1" H 8400 11600 50  0000 C CNN
-F 1 "10k" H 8400 11700 50  0000 C CNN
-F 2 "Resistor_SMD:R_0402_1005Metric" H 8250 11650 50  0001 C CNN
-F 3 "~" H 8250 11650 50  0001 C CNN
-	1    8250 11650
+P 5350 7350
+F 0 "R1" H 5500 7300 50  0000 C CNN
+F 1 "100k" H 5500 7400 50  0000 C CNN
+F 2 "Resistor_SMD:R_0402_1005Metric" H 5350 7350 50  0001 C CNN
+F 3 "~" H 5350 7350 50  0001 C CNN
+	1    5350 7350
 	1    0    0    -1
 $EndComp
@@
 	9100 12000 8100 12000
 Wire Wire Line
-	8250 11750 8250 12200
-Connection ~ 8250 12200
-Wire Wire Line
-	8250 12200 8100 12200
-Wire Wire Line
-	6800 11500 7500 11500
+	6350 11500 6750 11500
 Wire Wire Line
 	7500 11600 7500 11500
 Connection ~ 7500 11500
 Wire Wire Line
-	8250 11500 8250 11550
-Wire Wire Line
-	7500 11500 8250 11500
-Wire Wire Line
 	8550 11500 8550 11550
-Wire Wire Line
-	8250 11500 8550 11500
-Connection ~ 8250 11500
-$Comp
-L Connector_Generic:Conn_01x06 J11
-U 1 1 61D4C090
-P 10200 7650
-F 0 "J11" H 10280 7642 50  0000 L CNN
-F 1 "UART3_EXT" H 10280 7551 50  0000 L CNN
-F 2 "Connector_PinHeader_1.00mm:PinHeader_1x06_P1.00mm_Vertical" H 10200 7650 50  0001 C CNN
-F 3 "~" H 10200 7650 50  0001 C CNN
-	1    10200 7650
-	-1   0    0    -1
-$EndComp
 $Comp
 L power:GND #PWR0115
@@
 F 3 "" H 14050 12300 50  0001 C CNN
 	1    14050 12200
-	1    0    0    -1
+	1    0    0    1
 $EndComp
 Wire Wire Line
@@
 Wire Wire Line
 	20250 10250 19350 10250
+Wire Wire Line
+	10400 7950 10950 7950
+Text Label 10950 7950 2    39   ~ 0
+USART3_RX_NCP
+Text Label 10950 7850 2    39   ~ 0
+USART3_TX_NCP
+Wire Wire Line
+	10400 7850 10950 7850
+$Comp
+L Connector_Generic:Conn_01x06 J11
+U 1 1 61D4C090
+P 10200 7650
+F 0 "J11" H 10280 7642 50  0000 L CNN
+F 1 "UART3_EXT" H 10280 7551 50  0000 L CNN
+F 2 "Connector_PinHeader_1.00mm:PinHeader_1x06_P1.00mm_Vertical_SMD_Pin1Left" H 10200 7650 50  0001 C CNN
+F 3 "~" H 10200 7650 50  0001 C CNN
+	1    10200 7650
+	-1   0    0    -1
+$EndComp
+Wire Wire Line
+	10400 7750 10950 7750
+Text Label 10950 7750 2    39   ~ 0
+USART3_RTS_NCP
+Text Label 10950 7650 2    39   ~ 0
+USART3_CTS_NCP
+$Comp
+L Device:C_Small C20
+U 1 1 61D0B962
+P 19950 4050
+F 0 "C20" H 19858 4096 50  0000 R CNN
+F 1 "1u" H 19858 4005 50  0000 R CNN
+F 2 "Capacitor_SMD:C_0603_1608Metric" H 19950 4050 50  0001 C CNN
+F 3 "~" H 19950 4050 50  0001 C CNN
+	1    19950 4050
+	1    0    0    -1
+$EndComp
+Wire Wire Line
+	3150 9900 3150 10100
+Wire Wire Line
+	3550 9900 3650 9900
+Wire Wire Line
+	3650 9900 3650 9850
+Connection ~ 3550 9900
+$Comp
+L Device:C_Small C28
+U 1 1 61F7727F
+P 6750 11850
+F 0 "C28" H 6650 11750 50  0000 C CNN
+F 1 "0.1u" H 6600 11950 50  0000 C CNN
+F 2 "Capacitor_SMD:C_0402_1005Metric" H 6750 11850 50  0001 C CNN
+F 3 "~" H 6750 11850 50  0001 C CNN
+	1    6750 11850
+	-1   0    0    1
+$EndComp
+Wire Wire Line
+	6750 11750 6750 11500
+Connection ~ 6750 11500
+Wire Wire Line
+	6750 11500 7500 11500
+$Comp
+L power:GND #PWR0143
+U 1 1 62172771
+P 6750 12000
+F 0 "#PWR0143" H 6750 11750 50  0001 C CNN
+F 1 "GND" H 6755 11827 50  0001 C CNN
+F 2 "" H 6750 12000 50  0001 C CNN
+F 3 "" H 6750 12000 50  0001 C CNN
+	1    6750 12000
+	1    0    0    -1
+$EndComp
+Wire Wire Line
+	6750 12000 6750 11950
+Wire Wire Line
+	8100 12200 9100 12200
+Wire Wire Line
+	7500 11500 8550 11500
+Wire Wire Line
+	5350 7550 5350 7450
+Wire Wire Line
+	4350 7550 5350 7550
+Text Label 5850 7150 2    39   ~ 8
+VCC_MCU_3V3
+Wire Wire Line
+	5350 7250 5350 7150
+Wire Wire Line
+	5350 7150 5850 7150
+Wire Wire Line
+	18900 3850 19600 3850
+Wire Wire Line
+	18800 7050 19450 7050
+Wire Wire Line
+	15800 2400 16950 2400
 $EndSCHEMATC

Commit message: filling out layout
Parts:
- removed R23, R30: 0, Resistor_SMD:R_0402_1005Metric, symbol Device:R_Small
Connections:
- net STM_STATUS_0: now also J13.3 (Pin_3); no longer J13.5 (Pin_5)
- net STM_STATUS_L: now also J13.2 (Pin_2); no longer J13.3 (Pin_3)
- net STM_STATUS_R: now also J13.4 (Pin_4); no longer J13.7 (Pin_7)
- net SW_0: now also J13.7 (Pin_7); no longer J13.4 (Pin_4)
- net SW_L: now also J13.8 (Pin_8); no longer J13.2 (Pin_2)
- net SW_PWR: now also J13.5 (Pin_5); no longer J13.8 (Pin_8)
- no-connect marks 8 -> 10
Changed lines of the file:
@@
 Text Label 12250 6600 0    39   ~ 8
 VCC_BACKUP
-$Comp
-L Device:R_Small R30
-U 1 1 60A537BB
-P 13100 7650
-F 0 "R30" V 13050 7500 50  0000 C CNN
-F 1 "0" V 13050 7750 50  0000 C CNN
-F 2 "Resistor_SMD:R_0402_1005Metric" H 13100 7650 50  0001 C CNN
-F 3 "~" H 13100 7650 50  0001 C CNN
-	1    13100 7650
-	0    1    -1   0
-$EndComp
-Wire Wire Line
-	13200 7650 13500 7650
-$Comp
-L Device:R_Small R23
-U 1 1 60B2C13E
-P 13100 7550
-F 0 "R23" V 13050 7400 50  0000 C CNN
-F 1 "0" V 13050 7650 50  0000 C CNN
-F 2 "Resistor_SMD:R_0402_1005Metric" H 13100 7550 50  0001 C CNN
-F 3 "~" H 13100 7550 50  0001 C CNN
-	1    13100 7550
-	0    1    -1   0
-$EndComp
-Wire Wire Line
-	13200 7550 13500 7550
-Wire Wire Line
-	13000 7550 12250 7550
-Wire Wire Line
-	13000 7650 12250 7650
 NoConn ~ 14800 7650
 NoConn ~ 14800 7500
@@
 Text Label 12250 7400 0    39   ~ 0
 LPUART1_TX_GPS
-Text Label 12250 7550 0    39   ~ 0
-I2C4_SCL_SYSTEM
-Text Label 12250 7650 0    39   ~ 0
-I2C4_SDA_SYSTEM
 Wire Wire Line
 	13500 7850 13450 7850
@@
 Text Label 6250 9700 0    39   ~ 0
 SW_PWR_EXT
-Text Label 8850 10000 2    39   ~ 0
+Text Label 8850 9700 2    39   ~ 0
 SW_PWR
 Wire Wire Line
@@
 Wire Wire Line
 	6800 9300 6850 9300
-Wire Wire Line
-	8250 9800 8850 9800
-Wire Wire Line
-	8250 9600 8850 9600
-Wire Wire Line
-	8250 9400 8850 9400
-Wire Wire Line
-	8250 9900 8850 9900
-Wire Wire Line
-	8250 9700 8850 9700
-Wire Wire Line
-	8250 9500 8850 9500
-Text Label 8850 9400 2    39   ~ 0
+Text Label 8850 10000 2    39   ~ 0
 SW_L
-Text Label 8850 9600 2    39   ~ 0
+Text Label 8850 9900 2    39   ~ 0
 SW_0
 Text Label 8850 9800 2    39   ~ 0
 SW_R
-Text Label 8850 9900 2    39   ~ 0
+Text Label 8850 9600 2    39   ~ 0
 STM_STATUS_R
-Text Label 8850 9700 2    39   ~ 0
+Text Label 8850 9500 2    39   ~ 0
 STM_STATUS_0
-Text Label 8850 9500 2    39   ~ 0
+Text Label 8850 9400 2    39   ~ 0
 STM_STATUS_L
 Wire Wire Line
@@
 Wire Wire Line
 	15800 2400 16950 2400
+Wire Wire Line
+	8850 9400 8250 9400
+Wire Wire Line
+	8250 9500 8850 9500
+Wire Wire Line
+	8250 9600 8850 9600
+Wire Wire Line
+	8250 9700 8850 9700
+Wire Wire Line
+	8250 9800 8850 9800
+Wire Wire Line
+	8250 9900 8850 9900
+NoConn ~ 13500 7550
+NoConn ~ 13500 7650
 $EndSCHEMATC
