File: atlas_hw/atlas.sch (KiCad schematic (older format))
At the start: 169 parts, among them J1 USB_C_Receptacle_USB2.0, J10 PSP_LCD, J11 UART3_EXT, J12 IO_EXT, J13 IO_MAIN, J2 DEBUG_STM, J3 PSP_TOUCH, J4 UPDI_DSS, J5 CELL_THERM, J6 LPM027M128B, J7 FLEX_12380-03, J8 Micro_SD_Card_Det, J9 PSP_LCD_BL, Q1 Q_NMOS_DGS, Q2 Q_NMOS_DGS, Q4 Q_NMOS_DGS, Q5 Q_NMOS_DGS, SW1 BTN_L_EXT, SW2 BTN_0_EXT, SW3 ResetSTM, SW4 BTN_R_EXT, SW5 BTN_PWR_EXT, U1 STM32H723VITx, U10 BQ25611D, U11 L96-M33, U13 LSF0108, U14 NPP600SNADJ, U15 TPS61073, U16 PAM2841, U2 S27KL0641DABHV023, U3 MCP1811B, U4 TLV62569DBV, U5 MX25L3233FM2I-08G, U6 LC709203F, U7 ATtiny402-SS, U8 MS5637, U9 MC6470, Y1 16M, Y4 32k

Commit message: layout mostly done, split btn into diffrent file
Parts:
- removed C61: 0.1u, Capacitor_SMD:C_0402_1005Metric, symbol Device:C_Small
- removed R3: 0, Resistor_SMD:R_0402_1005Metric, symbol Device:R_Small
- added H1, H2, H3, H4: MountingHole_Pad, MountingHole:MountingHole_2.2mm_M2_Pad_Via, symbol Mechanical:MountingHole_Pad
- U10: footprint Package_DFN_QFN:WQFN-24-1EP_4x4mm_P0.5mm_EP2.7x2.7mm_ThermalVias -> Package_DFN_QFN:WQFN-24-1EP_4x4mm_P0.5mm_EP2.7x2.7mm
Connections:
- net labels removed: SPI4_FLASH_CS, SW_C
- wire segments 937 -> 939
Changed lines of the file:
@@
 F 0 "U10" H 11900 5700 50  0000 C CNN
 F 1 "BQ25611D" H 11900 5600 50  0000 C CNN
-F 2 "Package_DFN_QFN:WQFN-24-1EP_4x4mm_P0.5mm_EP2.7x2.7mm_ThermalVias" H 11600 5650 50  0001 C CNN
+F 2 "Package_DFN_QFN:WQFN-24-1EP_4x4mm_P0.5mm_EP2.7x2.7mm" H 11600 5650 50  0001 C CNN
 F 3 "http://www.ti.com/lit/ds/symlink/bq25601.pdf" H 11600 5900 50  0001 C CNN
 	1    11600 4500
@@
 Wire Wire Line
 	11100 3700 11050 3700
-$Comp
-L Device:R_Small R3
-U 1 1 688BA75A
-P 3500 4000
-F 0 "R3" V 3600 4100 50  0000 C CNN
-F 1 "0" V 3600 3900 50  0000 C CNN
-F 2 "Resistor_SMD:R_0402_1005Metric" H 3500 4000 50  0001 C CNN
-F 3 "~" H 3500 4000 50  0001 C CNN
-	1    3500 4000
-	0    -1   -1   0
-$EndComp
 Wire Wire Line
-	3400 4000 3250 4000
-Connection ~ 3250 4000
-Wire Wire Line
-	3750 4000 3750 4350
+	3750 4000 3750 4300
 $Comp
 L power:GND #PWR09
@@
 $EndComp
 Wire Wire Line
-	3600 4000 3750 4000
-Connection ~ 3750 4000
-Wire Wire Line
 	3750 4000 3900 4000
 Wire Wire Line
@@
 Wire Wire Line
 	15300 13700 15300 13850
-$Comp
-L Device:C_Small C61
-U 1 1 825AF0A3
-P 15400 11650
-F 0 "C61" H 15308 11696 50  0000 R CNN
-F 1 "0.1u" H 15308 11605 50  0000 R CNN
-F 2 "Capacitor_SMD:C_0402_1005Metric" H 15400 11650 50  0001 C CNN
-F 3 "~" H 15400 11650 50  0001 C CNN
-	1    15400 11650
-	1    0    0    -1
-$EndComp
-$Comp
-L power:GND #PWR0104
-U 1 1 8286616E
-P 15400 11800
-F 0 "#PWR0104" H 15400 11550 50  0001 C CNN
-F 1 "GND" H 15405 11627 50  0001 C CNN
-F 2 "" H 15400 11800 50  0001 C CNN
-F 3 "" H 15400 11800 50  0001 C CNN
-	1    15400 11800
-	1    0    0    -1
-$EndComp
-Wire Wire Line
-	15400 11800 15400 11750
 Wire Wire Line
 	15800 11500 15800 12250
 Wire Wire Line
-	15400 11500 15400 11550
-Wire Wire Line
 	15400 11500 15800 11500
 $Comp
@@
 	12100 2550 12100 3100
 Wire Wire Line
-	12300 2550 12300 3100
-Wire Wire Line
 	12300 2350 12300 2200
 Wire Wire Line
@@
 	12700 2800 13350 2800
 Wire Wire Line
-	11650 3000 13350 3000
+	11650 3000 12300 3000
 Wire Wire Line
 	15150 10250 15150 10400
@@
 	12500 2900 13350 2900
 Connection ~ 12100 3100
-Connection ~ 12300 3100
-Wire Wire Line
-	12300 3100 13350 3100
 Wire Wire Line
 	11550 3100 12100 3100
-Wire Wire Line
-	12100 3100 12300 3100
 Connection ~ 12300 2200
 Connection ~ 12700 2200
@@
 Wire Wire Line
 	7450 3600 7450 3650
-Text Label 5200 8150 2    39   ~ 0
+Text Label 5200 8350 2    39   ~ 0
 STM_STATUS_L
 Wire Wire Line
-	5200 8150 4350 8150
+	5200 8350 4350 8350
 Wire Wire Line
 	4350 8250 5200 8250
@@
 STM_STATUS_0
 Wire Wire Line
-	4350 8350 5200 8350
-Text Label 5200 8350 2    39   ~ 0
+	4350 8150 5200 8150
+Text Label 5200 8150 2    39   ~ 0
 STM_STATUS_R
 Wire Wire Line
-	4350 4650 5200 4650
+	4350 4750 5200 4750
 Wire Wire Line
-	4350 4950 5200 4950
+	4350 4650 5200 4650
+Text Label 5200 4750 2    39   ~ 0
+SW_0
 Text Label 5200 4650 2    39   ~ 0
-SW_C
-Text Label 5200 4950 2    39   ~ 0
 SW_R
 Wire Wire Line
@@
 ~USB_DET
 Wire Wire Line
-	4350 4750 5200 4750
-Text Label 5200 4750 2    39   ~ 0
+	4350 4950 5200 4950
+Text Label 5200 4950 2    39   ~ 0
 SW_L
 $Comp
@@
 	2300 14400 2850 14400
 Text Label 2300 14400 0    39   ~ 0
-SPI4_FLASH_CS
+SPI4_FLASH_NCS
 NoConn ~ 2850 14500
 NoConn ~ 2850 14600
@@
 NoConn ~ 13500 7550
 NoConn ~ 13500 7650
+Wire Wire Line
+	12100 3100 13350 3100
+Wire Wire Line
+	12300 2550 12300 3000
+Connection ~ 12300 3000
+Wire Wire Line
+	12300 3000 13350 3000
+Wire Wire Line
+	3650 4300 3750 4300
+Connection ~ 3650 4300
+Connection ~ 3750 4300
+Wire Wire Line
+	3750 4300 3750 4350
+$Comp
+L Mechanical:MountingHole_Pad H3
+U 1 1 613E3012
+P 8850 14150
+F 0 "H3" H 8950 14199 50  0000 L CNN
+F 1 "MountingHole_Pad" H 8950 14108 50  0000 L CNN
+F 2 "MountingHole:MountingHole_2.2mm_M2_Pad_Via" H 8850 14150 50  0001 C CNN
+F 3 "~" H 8850 14150 50  0001 C CNN
+	1    8850 14150
+	1    0    0    -1
+$EndComp
+$Comp
+L power:GND #PWR0104
+U 1 1 613F019F
+P 8850 14300
+F 0 "#PWR0104" H 8850 14050 50  0001 C CNN
+F 1 "GND" H 8855 14127 50  0001 C CNN
+F 2 "" H 8850 14300 50  0001 C CNN
+F 3 "" H 8850 14300 50  0001 C CNN
+	1    8850 14300
+	1    0    0    -1
+$EndComp
+Wire Wire Line
+	8850 14300 8850 14250
+$Comp
+L Mechanical:MountingHole_Pad H4
+U 1 1 616D581B
+P 8850 14600
+F 0 "H4" H 8950 14649 50  0000 L CNN
+F 1 "MountingHole_Pad" H 8950 14558 50  0000 L CNN
+F 2 "MountingHole:MountingHole_2.2mm_M2_Pad_Via" H 8850 14600 50  0001 C CNN
+F 3 "~" H 8850 14600 50  0001 C CNN
+	1    8850 14600
+	1    0    0    -1
+$EndComp
+$Comp
+L power:GND #PWR0144
+U 1 1 616D5821
+P 8850 14750
+F 0 "#PWR0144" H 8850 14500 50  0001 C CNN
+F 1 "GND" H 8855 14577 50  0001 C CNN
+F 2 "" H 8850 14750 50  0001 C CNN
+F 3 "" H 8850 14750 50  0001 C CNN
+	1    8850 14750
+	1    0    0    -1
+$EndComp
+Wire Wire Line
+	8850 14750 8850 14700
+$Comp
+L Mechanical:MountingHole_Pad H1
+U 1 1 617CCFBF
+P 8000 14150
+F 0 "H1" H 8100 14199 50  0000 L CNN
+F 1 "MountingHole_Pad" H 8100 14108 50  0000 L CNN
+F 2 "MountingHole:MountingHole_2.2mm_M2_Pad_Via" H 8000 14150 50  0001 C CNN
+F 3 "~" H 8000 14150 50  0001 C CNN
+	1    8000 14150
+	1    0    0    -1
+$EndComp
+$Comp
+L power:GND #PWR0145
+U 1 1 617CCFC5
+P 8000 14300
+F 0 "#PWR0145" H 8000 14050 50  0001 C CNN
+F 1 "GND" H 8005 14127 50  0001 C CNN
+F 2 "" H 8000 14300 50  0001 C CNN
+F 3 "" H 8000 14300 50  0001 C CNN
+	1    8000 14300
+	1    0    0    -1
+$EndComp
+Wire Wire Line
+	8000 14300 8000 14250
+$Comp
+L Mechanical:MountingHole_Pad H2
+U 1 1 618C4B9D
+P 8000 14600
+F 0 "H2" H 8100 14649 50  0000 L CNN
+F 1 "MountingHole_Pad" H 8100 14558 50  0000 L CNN
+F 2 "MountingHole:MountingHole_2.2mm_M2_Pad_Via" H 8000 14600 50  0001 C CNN
+F 3 "~" H 8000 14600 50  0001 C CNN
+	1    8000 14600
+	1    0    0    -1
+$EndComp
+$Comp
+L power:GND #PWR0146
+U 1 1 618C4BA3
+P 8000 14750
+F 0 "#PWR0146" H 8000 14500 50  0001 C CNN
+F 1 "GND" H 8005 14577 50  0001 C CNN
+F 2 "" H 8000 14750 50  0001 C CNN
+F 3 "" H 8000 14750 50  0001 C CNN
+	1    8000 14750
+	1    0    0    -1
+$EndComp
+Wire Wire Line
+	8000 14750 8000 14700
 $EndSCHEMATC

Commit message: atlas dev simplifcations
Parts:
- removed C31, C35, C47, C50: 1u, Capacitor_SMD:C_0603_1608Metric, symbol Device:C_Small
- removed C33: 0.1u, Capacitor_SMD:C_0402_1005Metric, symbol Device:C_Small
- removed C41: 47n, Capacitor_SMD:C_0402_1005Metric, symbol Device:C_Small
- removed C44: 4.7u, Capacitor_SMD:C_0603_1608Metric, symbol Device:C_Small
- removed D2: STM_STATUS_B, LED_SMD:LED_0805_2012Metric, symbol Device:LED_Small_ALT
- removed D5: CHARGE_STATUS, LED_SMD:LED_0805_2012Metric, symbol Device:LED_Small_ALT
- removed J1: USB_C_Receptacle_USB2.0, Connector_USB:USB_C_Receptacle_Amphenol_12401548E4-2A, symbol Connector:USB_C_Receptacle_USB2.0
- removed J11: UART3_EXT, Connector_PinHeader_1.00mm:PinHeader_1x06_P1.00mm_Vertical_SMD_Pin1Left, symbol Connector_Generic:Conn_01x06
- removed J12: IO_EXT, Connector_FFC-FPC:Hirose_FH12-10S-0.5SH_1x10-1MP_P0.50mm_Horizontal, symbol Connector_Generic:Conn_01x10
- removed J13: IO_MAIN, Connector_FFC-FPC:Hirose_FH12-10S-0.5SH_1x10-1MP_P0.50mm_Horizontal, symbol Connector_Generic:Conn_01x10
- removed J5: CELL_THERM, Connector_PinHeader_1.00mm:PinHeader_1x03_P1.00mm_Vertical, symbol Connector_Generic:Conn_01x03
- removed J6: LPM027M128B, Connector_FFC-FPC:Hirose_FH12-10S-0.5SH_1x10-1MP_P0.50mm_Horizontal, symbol Connector_Generic:Conn_01x10
- removed J7: FLEX_12380-03, Connector_PinHeader_1.00mm:PinHeader_1x02_P1.00mm_Vertical, symbol Connector_Generic:Conn_01x02
- removed L7: 1u, Inductor_SMD:L_Bourns-SRN4018, symbol Device:L_Small
- removed L9: L_Small, Inductor_SMD:L_Taiyo-Yuden_MD-3030, symbol Device:L_Small
- removed Q5: Q_NMOS_DGS, Package_TO_SOT_SMD:SOT-23, symbol Device:Q_NMOS_DGS
- removed R33, R35: 4.7k, Resistor_SMD:R_0402_1005Metric, symbol Device:R_Small
- removed R36, R41, R85, R86: 100k, Resistor_SMD:R_0402_1005Metric, symbol Device:R_Small
- removed R37: 1k, Resistor_SMD:R_0402_1005Metric, symbol Device:R_Small
- removed R49: 100, Resistor_SMD:R_0402_1005Metric, symbol Device:R_Small
- removed R56, R57: NP, Resistor_SMD:R_0402_1005Metric, symbol Device:R_Small
- removed U10: BQ25611D, Package_DFN_QFN:WQFN-24-1EP_4x4mm_P0.5mm_EP2.7x2.7mm, symbol atlas:BQ25611D
- removed U15: TPS61073, Package_TO_SOT_SMD:SOT-23-6, symbol atlas:TPS61070
- removed U6: LC709203F, atlas:WDFN-8_3x4mm_0.6mm_1.96x2.56mm, symbol atlas:LC709203F
- removed U8: MS5637, atlas:QFN-4_3x3_Pitch2mm, symbol atlas:MS5637
- added J1: USB_B_Micro, Connector_USB:USB_Micro-B_Molex-105017-0001, symbol Connector:USB_B_Micro
- added J5: EXP_L, Connector_PinHeader_2.54mm:PinHeader_1x18_P2.54mm_Vertical, symbol Connector_Generic:Conn_01x18
- added J6: EXP_R, Connector_PinHeader_2.54mm:PinHeader_1x18_P2.54mm_Vertical, symbol Connector_Generic:Conn_01x18
- added L1: 2.2u, Inductor_SMD:L_Bourns-SRN4018, symbol Device:L_Small
- added R2, R3: 100k, Resistor_SMD:R_0402_1005Metric, symbol Device:R_Small
- added R23, R30: NP, Resistor_SMD:R_0402_1005Metric, symbol Device:R_Small
- added U6: ST1PS02, atlas:TQFN-12_1.7x2.0mm_P0.4mm, symbol atlas:ST1PS02
- C12, C14, C4: value 4.7u -> 1u
- C15: value 4.7u -> 10u; footprint Capacitor_SMD:C_0603_1608Metric -> Capacitor_SMD:C_0805_2012Metric
- C16: value 4.7u -> 0.1u; footprint Capacitor_SMD:C_0603_1608Metric -> Capacitor_SMD:C_0402_1005Metric
- C18: value 0.1u -> 10u; footprint Capacitor_SMD:C_0402_1005Metric -> Capacitor_SMD:C_0603_1608Metric
- C5: value 0.1u -> 1u
- C9: value 1u -> 10u; footprint Capacitor_SMD:C_0603_1608Metric -> Capacitor_SMD:C_0805_2012Metric
- R10: value 1k -> 100k
- R12, R13: value 5.1k -> 0
- R17, R24: value 0 -> NP
- R31, R32: value 100k -> NP
Connections:
- net labels added: DSS_EXT, I2C4_SCL_SENSOR_PD12, I2C4_SDA_SENSOR_PD13, PA2, PA2_WKUP, PB6, PB7, PD15, PD6, PD7, PD9, PE0, PE1, SDMMC1_CKIN_PB8, SDMMC1_VSEL_PD1, SD_DET, SPI4_FLASH_NCS_PE4, SPI4_MISO_APP_PE5, SPI4_MOSI_APP_PE6, SPI4_SCK_APP_PE2, STM_VCORE_D0, STM_VCORE_D0_PB15, STM_VCORE_D1, STM_VCORE_D1_PB14, STM_VCORE_D2, STM_VCORE_D2_PB13, STM_VCORE_EN, STM_VCORE_EN_PB12, STM_VCORE_GOOD, STM_VCORE_GOOD_PD8, VCAP1, VCAP1_STM, VCAP2, VCAP2_STM, VCC_3V3, VCC_CORE, VCORE_EN
- net labels removed: BQ25611_INT, CELL_NEG, CELL_NTC, CELL_POS, CHG_STAT, EXTMODE, I2C4_SCL_SYSTEM, I2C4_SDA_SYSTEM, LC709203_INT, OPT_LCD_COM_INV, SPI4_OPT_LCD_NCS, STM_STATUS_0_EXT, STM_STATUS_B, STM_STATUS_L_EXT, STM_STATUS_R_EXT, SW_0_EXT, SW_L_EXT, SW_PWR_EXT, SW_R_EXT, USART3_CTS_NCP, USART3_RTS_NCP, USART3_RX_NCP, USART3_TX_NCP, USB_CHGR_D+, USB_CHGR_D-, VCC_3V3_EXT, VCC_LCD_PWR, ~USB_DET
- wire segments 939 -> 803
- no-connect marks 10 -> 11
Other:
- note removed: "4.8-5.2V"
- moved on the sheet: C10, C13, C27, C32, C34, C38, C48, C49, C52, C7, C8, D1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

Commit message: dfm reductions
Parts:
- removed C48: 1u, Capacitor_SMD:C_0603_1608Metric, symbol Device:C_Small
- removed C49, C59, C60: 0.1u, Capacitor_SMD:C_0402_1005Metric, symbol Device:C_Small
- removed C62, C63: 1u, Capacitor_SMD:C_0402_1005Metric, symbol Device:C_Small
- removed H1, H2, H3, H4: MountingHole_Pad, MountingHole:MountingHole_2.2mm_M2_Pad_Via, symbol Mechanical:MountingHole_Pad
- removed J4: UPDI_DSS, Connector_PinHeader_1.00mm:PinHeader_1x03_P1.00mm_Vertical, symbol Connector_Generic:Conn_01x03
- removed J5: EXP_L, Connector_PinHeader_2.54mm:PinHeader_1x18_P2.54mm_Vertical, symbol Connector_Generic:Conn_01x18
- removed J6: EXP_R, Connector_PinHeader_2.54mm:PinHeader_1x18_P2.54mm_Vertical, symbol Connector_Generic:Conn_01x18
- removed Q1, Q2, Q4: Q_NMOS_DGS, Package_TO_SOT_SMD:SOT-23, symbol Device:Q_NMOS_DGS
- removed R50: 100k, Resistor_SMD:R_0805_2012Metric, symbol Device:R_Small
- removed R54: 10k, Resistor_SMD:R_0402_1005Metric, symbol Device:R_Small
- removed R75: 200k, Resistor_SMD:R_0402_1005Metric, symbol Device:R_Small
- removed R76: 250k, Resistor_SMD:R_0402_1005Metric, symbol Device:R_Small
- removed R78, R79: 4.7k, Resistor_SMD:R_0402_1005Metric, symbol Device:R_Small
- removed U13: LSF0108, Package_DFN_QFN:WQFN-20-1EP_2.5x4.5mm_P0.5mm_EP1x2.9mm, symbol atlas:LSF0108
- removed U14: NPP600SNADJ, Package_SO:TSOP-5_1.65x3.05mm_P0.95mm, symbol atlas:NCP600SNADJ
- removed U16: PAM2841, Package_DFN_QFN:DFN-8-1EP_2x2mm_P0.5mm_EP0.9x1.5mm, symbol atlas:PAM2841
- removed U3: MCP1811B, Package_TO_SOT_SMD:SOT-23, symbol atlas:MCP1811B
- removed U7: ATtiny402-SS, Package_SO:SOIC-8_3.9x4.9mm_P1.27mm, symbol MCU_Microchip_ATtiny:ATtiny402-SS
- removed U9: MC6470, Package_LGA:LGA-12_2x2mm_P0.5mm, symbol atlas:MC6470
- added AE1: Antenna_Shield, Connector_Coaxial:U.FL_Hirose_U.FL-R-SMT-1_Vertical, symbol Device:Antenna_Shield
- added C29, C30, C31, C37, C42, C43, C44: 1u, Capacitor_SMD:C_0603_1608Metric, symbol Device:C_Small
- added C33, C39: 0.1u, Capacitor_SMD:C_0603_1608Metric, symbol Device:C_Small
- added C35, C36: 10u, Capacitor_SMD:C_0805_2012Metric, symbol Device:C_Small
- added C40: NP, Capacitor_SMD:C_0402_1005Metric, symbol Device:C_Small
- added C41: 4.7u, Capacitor_SMD:C_0603_1608Metric, symbol Device:C_Small
- added D11: MBR0540, Diode_SMD:D_SOD-123, symbol Device:D_Schottky_Small_ALT
- added D2: GPS_3DF, LED_SMD:LED_0805_2012Metric, symbol Device:LED_Small_ALT
- added D5: GPS_JAM, LED_SMD:LED_0805_2012Metric, symbol Device:LED_Small_ALT
- added H1, H2, H3, H4: MountingHole, MountingHole:MountingHole_2.7mm_M2.5, symbol Mechanical:MountingHole
- added J5: CELL, symbol Connector_Generic:Conn_01x03
- added J6: EXT, symbol Connector_Generic:Conn_02x15_Counter_Clockwise
- added J7: Conn_02x10_Counter_Clockwise, symbol Connector_Generic:Conn_02x10_Counter_Clockwise
- added JP1: GPS_EXT, symbol Jumper:Jumper_3_Bridged12
- added L2, L4: 2.2u, Inductor_SMD:L_Wuerth_MAPI-2510, symbol Device:L_Small
- added L5: 47n, Inductor_SMD:L_Wuerth_MAPI-2510, symbol Device:L_Small
- added R33, R41: 0, Resistor_SMD:R_0603_1608Metric, symbol Device:R_Small
- added R35, R36, R46, R49: 100k, Resistor_SMD:R_0603_1608Metric, symbol Device:R_Small
- added R37: 440k, Resistor_SMD:R_0603_1608Metric, symbol Device:R_Small
- added SW6: BTN_BOOT, Button_Switch_SMD:SW_SPST_PTS810, symbol Switch:SW_Push
- added TP1: VCC_CORE, symbol Connector:TestPoint
- added TP2: VCORE_FLAG, symbol Connector:TestPoint
- added TP3: PERIPH_FLAG, symbol Connector:TestPoint
- added U10: MAX17048, Package_DFN_QFN:DFN-8-1EP_2x2mm_P0.5mm_EP0.9x1.5mm, symbol atlas:MAX17048
- added U12: LV52204MU, Package_DFN_QFN:DFN-6-1EP_2x2mm_P0.65mm_EP1x1.6mm, symbol atlas:LV52204MU
- added U13: AP22804, Package_DFN_QFN:DFN-6-1EP_2x2mm_P0.65mm_EP1x1.6mm, symbol atlas:AP22804
- added U3, U7: MCP1810, Package_DFN_QFN:DFN-8-1EP_2x2mm_P0.5mm_EP0.9x1.5mm, symbol atlas:MCP1810
- added U8: MCP1640B, Package_TO_SOT_SMD:SOT-23-6, symbol atlas:TPS61070
- added U9: BQ25606, Package_DFN_QFN:WQFN-24-1EP_4x4mm_P0.5mm_EP2.7x2.7mm, symbol atlas:BQ25606
- C1, C11, C16, C17, C2, C22, C23, C24, C25, C26, C3, C38, C54, C56, C57, C58, C6: footprint Capacitor_SMD:C_0402_1005Metric -> Capacitor_SMD:C_0603_1608Metric
- C18: footprint Capacitor_SMD:C_0603_1608Metric -> Capacitor_SMD:C_0805_2012Metric
- C19, C21: value 22p -> 18p; footprint Capacitor_SMD:C_0402_1005Metric -> Capacitor_SMD:C_0603_1608Metric
- C28: value 0.1u -> NP
- C32: value 0.1u -> 10u; footprint Capacitor_SMD:C_0402_1005Metric -> Capacitor_SMD:C_0805_2012Metric
- C34: value 0.1u -> 4.7u; footprint Capacitor_SMD:C_0402_1005Metric -> Capacitor_SMD:C_0805_2012Metric
- C7: value 10u -> 4.7u
- C8: value 1u -> 4.7u
- D3: value GPS_3DF -> CHG_STATUS
- D6: value D_Schottky_Small_ALT -> MBR0540; footprint Diode_SMD:D_SOD-110 -> Diode_SMD:D_SOD-123
- J1: footprint Connector_USB:USB_Micro-B_Molex-105017-0001 -> Connector_USB:USB_Micro-B_Molex_47346-0001
- J10: footprint Connector_FFC-FPC:Hirose_FH12-40S-0.5SH_1x40-1MP_P0.50mm_Horizontal -> (none); Order No (none) -> 2135964; Price (none) -> 0.7248
- J2: Order No (none) -> 2886068; Price (none) -> 0.564
- J3: footprint Connector_FFC-FPC:Hirose_FH12-6S-0.5SH_1x06-1MP_P0.50mm_Horizontal -> (none); Order No (none) -> 2946022; Price (none) -> 0.1248
- J8: footprint Connector_Card:microSD_HC_Hirose_DM3BT-DSF-PEJS -> (none)
- J9: footprint atlas:Kyocera_046298_004_1x04_P0.5mm_Bottom -> (none); Order No (none) -> 2328702; Price (none) -> 0.1212
- L1: footprint Inductor_SMD:L_Bourns-SRN4018 -> Inductor_SMD:L_Wuerth_MAPI-2510; Order No (none) -> 2917560; Price (none) -> 0.2460
- L10: value 3.9n -> 22u; footprint Inductor_SMD:L_Taiyo-Yuden_MD-3030 -> Inductor_SMD:L_Bourns-SRN4018; Order No (none) -> 2616895; Price (none) -> 0.4428
- L3: value L_Small -> 2.2u; footprint Inductor_SMD:L_Bourns-SRN4018 -> Inductor_SMD:L_Wuerth_MAPI-2510; Order No (none) -> 2917560; Price (none) -> 0.2460
- R1: value 100k -> 0; footprint Resistor_SMD:R_0402_1005Metric -> Resistor_SMD:R_0805_2012Metric
- R10: value 100k -> NP; footprint Resistor_SMD:R_0402_1005Metric -> Resistor_SMD:R_0603_1608Metric
- R11, R18, R19, R40, R45, R48: footprint Resistor_SMD:R_0805_2012Metric -> Resistor_SMD:R_0603_1608Metric
- R12, R13, R14, R15, R16, R17, R21, R23, R24, R25, R30, R31, R32, R34, R42, R47, R5, R55, R7, R8, R82, R83, R84, R87, R9: footprint Resistor_SMD:R_0402_1005Metric -> Resistor_SMD:R_0603_1608Metric
- R2, R6: value 100k -> 1k; footprint Resistor_SMD:R_0402_1005Metric -> Resistor_SMD:R_0603_1608Metric
- R20: footprint Resistor_SMD:R_0603_1608Metric -> Resistor_SMD:R_0805_1608Metric
- R22: value 0 -> 100k; footprint Resistor_SMD:R_0402_1005Metric -> Resistor_SMD:R_0603_1608Metric
- R26: value NP -> 450; footprint Resistor_SMD:R_0402_1005Metric -> Resistor_SMD:R_0603_1608Metric
- R27: value NP -> 240; footprint Resistor_SMD:R_0402_1005Metric -> Resistor_SMD:R_0603_1608Metric
- R28, R29: value 4.7k -> 5.7k; footprint Resistor_SMD:R_0402_1005Metric -> Resistor_SMD:R_0603_1608Metric
- R3, R43: value 100k -> 0; footprint Resistor_SMD:R_0402_1005Metric -> Resistor_SMD:R_0603_1608Metric
- R38: value 100k -> 5.7k; footprint Resistor_SMD:R_0402_1005Metric -> Resistor_SMD:R_0603_1608Metric
- R39: value 0 -> 30k; footprint Resistor_SMD:R_0402_1005Metric -> Resistor_SMD:R_0603_1608Metric
- R4: value 200k -> 100k; footprint Resistor_SMD:R_0402_1005Metric -> Resistor_SMD:R_0603_1608Metric
- R44: value 100k -> 10; footprint Resistor_SMD:R_0402_1005Metric -> Resistor_SMD:R_0603_1608Metric
- RN1, RN2, RN3, RN4: Order No (none) -> 9235469; Price (none) -> 0.0466
- SW1: value BTN_L_EXT -> BTN_L; footprint Button_Switch_SMD:SW_SPST_B3S-1000 -> Button_Switch_SMD:SW_SPST_PTS645
- SW2: value BTN_0_EXT -> BTN_0; footprint Button_Switch_SMD:SW_SPST_B3S-1000 -> Button_Switch_SMD:SW_SPST_PTS645
- SW3: footprint Jumper:SolderJumper-2_P1.3mm_Open_Pad1.0x1.5mm -> Button_Switch_SMD:SW_SPST_PTS810; Order No (none) -> 3023215; Price (none) -> 0.1812
- SW4: value BTN_R_EXT -> BTN_R; footprint Button_Switch_SMD:SW_SPST_B3S-1000 -> Button_Switch_SMD:SW_SPST_PTS645
- SW5: value BTN_PWR_EXT -> BTN_PWR; footprint Button_Switch_SMD:SW_SPST_B3U-1000P -> Button_Switch_SMD:SW_SPST_PTS810; Order No (none) -> 3023215; Price (none) -> 0.1812
- U1: value STM32H723VITx -> STM32H723VGT6; Order No (none) -> 3576957; Price (none) -> 10.656
- U11: Price (none) -> 10.50
- U2: Order No (none) -> 2749802; Price (none) -> 1.44
- U4: Order No (none) -> 3121687; Price (none) -> 0.5820
- U5: Order No (none) -> 3129177; Price (none) -> 0.7116
- U6: Order No (none) -> 3527118; Price (none) -> 1.224
- Y1: value 16M -> 8M; Order No (none) -> 2854268; Price (none) -> 0.7248
- Y4: Order No (none) -> 3228354; Price (none) -> 0.3948
Connections:
- net labels added: BL_HV, CELL_NTC, CELL_POS, CHG_STATUS, FUEL_INT, GPS_INT, GPS_JAM, I2C4_SCL_SENSOR_PB6, I2C4_SCL_SENSOR_PB7, LCD_REG_EN, MCU_3V3_EN, PD13, PD4, PD5, PERIPH_FLG, PERIPH_REG_EN, STM_STATUS_C, SW_BOOT, SW_C, TOUCH_INT, USART3_CTS_NCP_PD11, USART3_RTS_NCP_PD12, USART3_RX_NCP_PD9, USART3_TX_NCP_PD8, USB_CHG_D+, USB_CHG_D-, VCC_3V3_MCU, VCC_3V3_MCU_EN, VCC_3V3_PERIPH, VCC_LCD_PWR, ~USB_DET
- net labels removed: DSS_EXT, EN_LCD_PWR, I2C1_SCL_SENSOR, I2C1_SDA_SENSOR, I2C4_SCL_SENSOR_PD12, I2C4_SDA_SENSOR_PD13, MC6470_INTA, MC6470_INTM, PA2, PA2_WKUP, PB6, PB7, PD15, PD6, PD7, PD9, PWR_ACK_DSS, PWR_EN_O, PWR_SW_DSS, SDMMC1_CKIN, SDMMC1_VSEL, SPI4_FLASH_NCS_PE4, STC911_INT, STC911_RESET, STM_STATUS_0, STM_VCORE_D0_PB15, STM_VCORE_D1_PB14, STM_VCORE_D2_PB13, STM_VCORE_EN_PB12, STM_VCORE_GOOD_PD8, SW_0, UDPI_DSS, VCORE_EN, VDD_SD_IO_3V3_1V8
- wire segments 803 -> 856
- no-connect marks 11 -> 10
Other:
- note removed: "0 = 1.8V\n1 = 3.3V"
- note removed: "NPP600 should maintain low Iq in dropout."
- moved on the sheet: C1, C10, C11, C12, C13, C14, C15, C16, C17, C18, C19, C2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

Commit message: lots of modifications to sch and board
Parts:
- removed J6: EXT, symbol Connector_Generic:Conn_02x15_Counter_Clockwise
- removed JP1: GPS_EXT, symbol Jumper:Jumper_3_Bridged12
- removed TP2: VCORE_FLAG, symbol Connector:TestPoint
- removed TP3: PERIPH_FLAG, symbol Connector:TestPoint
- added C45: 10u, Capacitor_SMD:C_0805_2012Metric, symbol Device:C_Small
- added C46, C47, C48, C59, C60, C61, C63, C64, C65: 0.1u, Capacitor_SMD:C_0402_1005Metric, symbol Device:C_Small
- added C49, C50, C55: 1u, Capacitor_SMD:C_0603_1608Metric, symbol Device:C_Small
- added C62: 10n, Capacitor_SMD:C_0402_1005Metric, symbol Device:C_Small
- added J4: DEBUG_NCP, Connector_PinHeader_1.27mm:PinHeader_2x05_P1.27mm_Vertical_SMD, symbol Connector_Generic:Conn_02x05_Odd_Even
- added JP2: Jumper_NO_Small, Connector_PinHeader_1.00mm:PinHeader_1x02_P1.00mm_Vertical, symbol Device:Jumper_NO_Small
- added L6: FERRITE, Inductor_SMD:L_0603_1608Metric, symbol Device:L_Small
- added R50, R51: 0, Resistor_SMD:R_0402_1005Metric, symbol Device:R_Small
- added RV1: 200k, Potentiometer_SMD:Potentiometer_Bourns_3314J_Vertical, symbol Device:R_POT
- added SW7: NP, Button_Switch_SMD:SW_SPST_PTS645, symbol Switch:SW_Push
- added U14: MS5637, atlas:QFN-4_3x3_Pitch2mm, symbol atlas:MS5637
- added U15: SHT4x, atlas:SHT_QFN-4-1EP_1.5x1.5mm, symbol atlas:SHT4x
- added U16: PSP_JOY, atlas:PSP-JOY, symbol atlas:PSP_JOY
- added U17: BGM220P, atlas:BGM220P, symbol atlas:BGM220P
- added U18: FXOS8700CQ, atlas:LGA-16_3x3mm_P0.5mm_LayoutBorder3x5y, symbol atlas:FXOS8700CQ
- added U19: L2G2IS, atlas:LGA-16_2.3x2.3mm_P0.4mm_LayoutBorder3x5y, symbol atlas:L2G2IS
- added U20: AZ2117, Package_TO_SOT_SMD:SOT-223-3_TabPin2, symbol Regulator_Linear:NCP1117-12_SOT223
- C11, C16, C17, C2, C22, C23, C24, C25, C26, C33, C38, C39, C54, C56, C57, C58, C6: footprint Capacitor_SMD:C_0603_1608Metric -> Capacitor_SMD:C_0402_1005Metric
- C29, C44: value 1u -> 10u; footprint Capacitor_SMD:C_0603_1608Metric -> Capacitor_SMD:C_0805_2012Metric
- C30: value 1u -> 0.1u; footprint Capacitor_SMD:C_0603_1608Metric -> Capacitor_SMD:C_0402_1005Metric
- C31: value 1u -> 4.7u; footprint Capacitor_SMD:C_0603_1608Metric -> Capacitor_SMD:C_0805_2012Metric
- C41, C8: footprint Capacitor_SMD:C_0603_1608Metric -> Capacitor_SMD:C_0805_2012Metric
- D5: value GPS_JAM -> NP
- D9: value STM_STATUS_0 -> PERIPH_FAULT
- H1, H2, H3, H4: footprint MountingHole:MountingHole_2.7mm_M2.5 -> MountingHole:MountingHole_2.7mm_M2.5_Pad_Via; symbol Mechanical:MountingHole -> Mechanical:MountingHole_Pad
- J10: footprint (none) -> Connector_FFC-FPC:Hirose_FH12-40S-0.5SH_1x40-1MP_P0.50mm_Horizontal
- J5: footprint (none) -> Connector_PinHeader_1.27mm:PinHeader_1x03_P1.27mm_Vertical
- L5: footprint Inductor_SMD:L_Wuerth_MAPI-2510 -> Inductor_SMD:L_0402_1005Metric
- R1: value 0 -> 1k; footprint Resistor_SMD:R_0805_2012Metric -> Resistor_SMD:R_0603_1608Metric
- R16: value 0 -> 100k
- R18: value 1k -> NP
- R20: footprint Resistor_SMD:R_0805_1608Metric -> Resistor_SMD:R_0603_1608Metric
- R26: value 450 -> 1k
- R27: value 240 -> 1k
- R28, R29, R38: value 5.7k -> 5.23k
- R33: value 0 -> NP
- R35: value 100k -> 316k
- R46: value 100k -> 0; footprint Resistor_SMD:R_0603_1608Metric -> Resistor_SMD:R_0402_1005Metric
- R7: value 1k -> 100k
- SW2: value BTN_0 -> ResetNCP; Order No (none) -> 3023215; Price (none) -> 0.1812
- SW3, SW5, SW6: footprint Button_Switch_SMD:SW_SPST_PTS810 -> Button_Switch_SMD:SW_SPST_PTS645
- TP1: footprint (none) -> TestPoint:TestPoint_Bridge_Pitch2.0mm_Drill0.7mm; symbol Connector:TestPoint -> Connector:TestPoint_2Pole
Connections:
- net labels added: ACCEL_INT1, ACCEL_INT2, DEBUG_NRESET_NCP, DEBUG_SWDCLK_NCP, DEBUG_SWDIO_NCP, DEBUG_SWO_NCP, GYRO_INT, I2C4_SCL_SENSOR, I2C4_SDA_SENSOR, I2C4_SDA_SENSOR_PB7, JOY_X, JOY_Y, PERIPH_FAULT, PTI_DATA, PTI_FRAME, SPI4_ACCEL_NCS, SPI4_GYRO_NCS, SPI4_NCS_ACCEL, SPI4_NCS_GYRO, USART3_CTS_NCP, USART3_RTS_NCP, USART3_RX_NCP, USART3_TX_NCP
- net labels removed: GPS_JAM, I2C4_SCL_SENSOR_PB7, PD13, PD4, PD5, PE0, PE1, PERIPH_FLG, SPI4_MISO_APP_PE5, SPI4_MOSI_APP_PE6, SPI4_SCK_APP_PE2, STM_STATUS_C, SW_C, USART3_CTS_NCP_PD11, USART3_RTS_NCP_PD12, USART3_RX_NCP_PD9, USART3_TX_NCP_PD8
- wire segments 856 -> 958
- no-connect marks 10 -> 11
Other:
- note added: "Test Regulator - 2.5-5V @ 1A"
- moved on the sheet: AE1, C2, C20, C28, C32, C33, C34, C35, C36, C37, C38, C39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
