File: atlas_hw/atlas.sch (KiCad schematic (older format))
At the start: 189 parts, among them J1 USB_B_Micro, J10 PSP_LCD, J2 DEBUG_STM, J3 PSP_TOUCH, J4 DEBUG_NCP, J5 CELL, J7 Conn_02x10_Counter_Clockwise, J8 Micro_SD_Card_Det, J9 PSP_LCD_BL, SW1 BTN_L, SW2 ResetNCP, SW3 ResetSTM, SW4 BTN_R, SW5 BTN_PWR, SW6 BTN_BOOT, SW7 NP, U1 STM32H723VGT6, U10 MAX17048, U11 L96-M33, U12 LV52204MU, U13 AP22804, U14 MS5637, U15 SHT4x, U16 PSP_JOY, U17 BGM220P, U18 FXOS8700CQ, U19 L2G2IS, U2 S27KL0641DABHV023, U20 AZ2117, U3 MCP1810, U4 TLV62569DBV, U5 MX25L3233FM2I-08G, U6 ST1PS02, U7 MCP1810, U8 MCP1640B, U9 BQ25606, Y1 8M, Y4 32k

Commit message: final component placement
Parts:
- removed C28, C40: NP, Capacitor_SMD:C_0402_1005Metric, symbol Device:C_Small
- removed C41: 4.7u, Capacitor_SMD:C_0805_2012Metric, symbol Device:C_Small
- removed C42, C43, C49, C55: 1u, Capacitor_SMD:C_0603_1608Metric, symbol Device:C_Small
- removed C44: 10u, Capacitor_SMD:C_0805_2012Metric, symbol Device:C_Small
- removed C47, C48, C60, C64: 0.1u, Capacitor_SMD:C_0402_1005Metric, symbol Device:C_Small
- removed C62: 10n, Capacitor_SMD:C_0402_1005Metric, symbol Device:C_Small
- removed H1, H2: MountingHole, MountingHole:MountingHole_2.7mm_M2.5_Pad_Via, symbol Mechanical:MountingHole_Pad
- removed J4: DEBUG_NCP, Connector_PinHeader_1.27mm:PinHeader_2x05_P1.27mm_Vertical_SMD, symbol Connector_Generic:Conn_02x05_Odd_Even
- removed J7: Conn_02x10_Counter_Clockwise, symbol Connector_Generic:Conn_02x10_Counter_Clockwise
- removed J8: Micro_SD_Card_Det, symbol Connector:Micro_SD_Card_Det
- removed JP2: Jumper_NO_Small, Connector_PinHeader_1.00mm:PinHeader_1x02_P1.00mm_Vertical, symbol Device:Jumper_NO_Small
- removed L6: FERRITE, Inductor_SMD:L_0603_1608Metric, symbol Device:L_Small
- removed R14, R15, R21: 0, Resistor_SMD:R_0603_1608Metric, symbol Device:R_Small
- removed R16, R22, R34, R45: 100k, Resistor_SMD:R_0603_1608Metric, symbol Device:R_Small
- removed R17, R23, R24, R30, R31, R32: NP, Resistor_SMD:R_0603_1608Metric, symbol Device:R_Small
- removed R50: 0, Resistor_SMD:R_0402_1005Metric, symbol Device:R_Small
- removed RV1: 200k, Potentiometer_SMD:Potentiometer_Bourns_3314J_Vertical, symbol Device:R_POT
- removed SW2: ResetNCP, Button_Switch_SMD:SW_SPST_PTS645, symbol Switch:SW_Push
- removed TP1: VCC_CORE, TestPoint:TestPoint_Bridge_Pitch2.0mm_Drill0.7mm, symbol Connector:TestPoint_2Pole
- removed U13: AP22804, Package_DFN_QFN:DFN-6-1EP_2x2mm_P0.65mm_EP1x1.6mm, symbol atlas:AP22804
- removed U15: SHT4x, atlas:SHT_QFN-4-1EP_1.5x1.5mm, symbol atlas:SHT4x
- removed U16: PSP_JOY, atlas:PSP-JOY, symbol atlas:PSP_JOY
- removed U17: BGM220P, atlas:BGM220P, symbol atlas:BGM220P
- removed U19: L2G2IS, atlas:LGA-16_2.3x2.3mm_P0.4mm_LayoutBorder3x5y, symbol atlas:L2G2IS
- removed U20: AZ2117, Package_TO_SOT_SMD:SOT-223-3_TabPin2, symbol Regulator_Linear:NCP1117-12_SOT223
- removed U7: MCP1810, Package_DFN_QFN:DFN-8-1EP_2x2mm_P0.5mm_EP0.9x1.5mm, symbol atlas:MCP1810
- added J6: 47352-1001, atlas:MOLEX_47352-1001, symbol atlas:47352-1001
- added J7: DEBUG_STM, Connector_PinHeader_1.27mm:PinHeader_2x05_P1.27mm_Vertical_SMD, symbol atlas:Conn_ARM_JTAG_SWD_10
- added Q1: DMC2990UDJ, Package_TO_SOT_SMD:SOT-363_SC-70-6, symbol atlas:Q_DUAL_NMOS_PMOS
- added U7: EYSHSNZWZ, atlas:XCVR_EYSHSNZWZ, symbol atlas:EYSHSNZWZ
- D5: value NP -> STM_STATUS_C
- D9: value PERIPH_FAULT -> NCP_STATUS
- J10: footprint Connector_FFC-FPC:Hirose_FH12-40S-0.5SH_1x40-1MP_P0.50mm_Horizontal -> atlas:J_SMD_4-1734839-0-40_0.5_25.43_5.1_2.05
- J3: footprint (none) -> atlas:TE_2328702-6
- J5: footprint Connector_PinHeader_1.27mm:PinHeader_1x03_P1.27mm_Vertical -> Connector_PinHeader_1.00mm:PinHeader_1x03_P1.00mm_Vertical
- R1: value 1k -> 10k; footprint Resistor_SMD:R_0603_1608Metric -> Resistor_SMD:R_0402_1005Metric
- R10: value NP -> 1k
- R18: value NP -> 1l
- R3: value 0 -> 100k
- R33: value NP -> 100k
- R82, R83, R84: footprint Resistor_SMD:R_0603_1608Metric -> Jumper:SolderJumper-2_P1.3mm_Open_TrianglePad1.0x1.5mm
- SW1, SW3, SW4: footprint Button_Switch_SMD:SW_SPST_PTS645 -> Button_Switch_SMD:SW_SPST_PTS810
- SW2: renamed from SW6; footprint Button_Switch_SMD:SW_SPST_PTS645 -> Button_Switch_SMD:SW_SPST_PTS810
- SW5: value BTN_PWR -> ResetNCP; footprint Button_Switch_SMD:SW_SPST_PTS645 -> Button_Switch_SMD:SW_SPST_PTS810
- SW7: value NP -> BTN_C; footprint Button_Switch_SMD:SW_SPST_PTS645 -> Button_Switch_SMD:SW_SPST_PTS810
- Y1: symbol Device:Crystal_Small -> Device:Crystal_GND24_Small
- Y4: footprint Crystal:Crystal_SMD_3215-2Pin_3.2x1.5mm -> Crystal:Crystal_SMD_MicroCrystal_CC7V-T1A-2Pin_3.2x1.5mm
Connections:
- net labels added: NCP_STATUS, SDMMC1_CKIN, SD_VSEL, STM_STATUS_C, SW_C_PWR, T2C4_LCD_BL
- net labels removed: GPS_EXTINT, I2C4_SCL_SENSOR_PB6, I2C4_SDA_SENSOR_PB7, PERIPH_FAULT, PERIPH_REG_EN, PTI_DATA, PTI_FRAME, SDMMC1_CKIN_PB8, SDMMC1_DET, SDMMC1_VSEL_PD1, SD_CLK, SD_CMD, SD_D0, SD_D1, SD_D2, SD_D3, SPI4_NCS_ACCEL, SPI4_NCS_GYRO, T3C1_LCD_BL, VCAP1_STM, VCAP2_STM, VCC_3V3_MCU_EN, VCC_3V3_PERIPH
- wire segments 958 -> 812
Other:
- note removed: "Test Regulator - 2.5-5V @ 1A"
- moved on the sheet: AE1, C1, C10, C11, C12, C13, C14, C15, C16, C17, C19, C2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

Commit message: layout done
Parts:
- removed C51: 10u, Capacitor_SMD:C_0805_2012Metric, symbol Device:C_Small
- removed D9: NCP_STATUS, LED_SMD:LED_0805_2012Metric, symbol Device:LED_Small_ALT
- removed J10: PSP_LCD, atlas:J_SMD_4-1734839-0-40_0.5_25.43_5.1_2.05, symbol Connector_Generic:Conn_01x40
- removed J7: DEBUG_STM, Connector_PinHeader_1.27mm:PinHeader_2x05_P1.27mm_Vertical_SMD, symbol atlas:Conn_ARM_JTAG_SWD_10
- removed R10: 1k, Resistor_SMD:R_0603_1608Metric, symbol Device:R_Small
- added BZ1: Buzzer, atlas:PKLCS1212, symbol Device:Buzzer
- added C28: 1u, Capacitor_SMD:C_0603_1608Metric, symbol Device:C_Small
- added C40, C41: 18p, Capacitor_SMD:C_0402_1005Metric, symbol Device:C_Small
- added C42: 0.1u, Capacitor_SMD:C_0402_1005Metric, symbol Device:C_Small
- added D12: NCP_0, LED_SMD:LED_0805_2012Metric, symbol Device:LED_Small_ALT
- added H1, H2: MountingHole, MountingHole:MountingHole_2.7mm_M2.5_Pad_Via, symbol Mechanical:MountingHole_Pad
- added J4: DEBUG_NCP, Connector_PinHeader_1.27mm:PinHeader_2x05_P1.27mm_Vertical_SMD, symbol atlas:Conn_ARM_JTAG_SWD_10
- added J7: Conn_01x40_Shielded, atlas:J_SMD_4-1734839-0-40_0.5_25.43_5.1_2.05, symbol Connector_Generic_Shielded:Conn_01x40_Shielded
- added Q2: Q_NPN_BCE, Package_TO_SOT_SMD:SOT-23, symbol Device:Q_NPN_BCE
- added R14: 0, Jumper:SolderJumper-2_P1.3mm_Open_TrianglePad1.0x1.5mm, symbol Device:R_Small
- added R15: NP, Jumper:SolderJumper-2_P1.3mm_Open_TrianglePad1.0x1.5mm, symbol Device:R_Small
- added R21: 100k, Resistor_SMD:R_0603_1608Metric, symbol Device:R_Small
- added R22: 1k, Resistor_SMD:R_0603_1608Metric, symbol Device:R_Small
- added Y2: 32k, Crystal:Crystal_SMD_MicroCrystal_CC7V-T1A-2Pin_3.2x1.5mm, symbol Device:Crystal_Small
- C1, C19, C21, C3: footprint Capacitor_SMD:C_0603_1608Metric -> Capacitor_SMD:C_0402_1005Metric
- J9: footprint (none) -> atlas:SFV4R-1STE1LF
- R12, R13: footprint Resistor_SMD:R_0603_1608Metric -> Jumper:SolderJumper-2_P1.3mm_Open_TrianglePad1.0x1.5mm
- R7: value 100k -> 1k
- R82, R83, R84: footprint Jumper:SolderJumper-2_P1.3mm_Open_TrianglePad1.0x1.5mm -> Resistor_SMD:R_0402_1005Metric
- U7: footprint atlas:XCVR_EYSHSNZWZ -> XCVR_EYSHSNZWZ
Connections:
- net GYRO_INT is gone; now on net FUEL_INT: U1.90 (PB4)
- net JOY_X is gone; now on net SW_C_PWR: U1.22 (PA0)
- net JOY_Y is gone; now on net SW_R: U1.23 (PA1)
- net SDMMC1_CKIN is gone; now on net GPS_FORCEON: U1.95 (PB8)
- net SPI4_GYRO_NCS is gone; now on net GPS_UART8_TX: U1.98 (PE1)
- net SW_PWR is gone; now on net TOUCH_INT: U1.7 (PC13)
- net VCC_3V3 is gone; now on net VCC_3V3_MCU: R28.1, R29.1, R42.1, R49.1
- net VCC_MCU_3V3 is gone; now on net VCC_3V3_MCU: SW1.1, SW2.1, SW4.1, SW7.1
- net ACCEL_INT1: now also U1.87 (PD6); no longer U1.86 (PD5)
- net ACCEL_INT2: now also U1.88 (PD7); no longer U1.85 (PD4)
- net BL_HV: now also J9.1 (Pin_1); no longer J9.4 (Pin_4)
- net DEBUG_NRESET_NCP: now also U7.19 (P0.21/RESET), J4.10 (~RESET~), R21.1; no longer R7.1, U7.25 (P0.20/TRACECLK)
- net DEBUG_NRESET_STM: no longer U2.A4 (RESET#)
- net DEBUG_SWDCLK_NCP: now also J4.4 (SWDCLK)
- net DEBUG_SWDIO_NCP: now also J4.2 (SWDIO)
- net DEBUG_SWO_NCP: now also U7.22 (P0.18/TRACEDATA[0]), J4.6 (SWO)
- net FUEL_INT: no longer U1.87 (PD6)
- net GND: now also RN1.1 (R1.1), RN1.2 (R2.1), RN1.3 (R3.1), RN1.4 (R4.1), RN2.1 (R1.1), RN2.2 (R2.1), RN2.3 (R3.1), RN2.4 (R4.1), RN3.1 (R1.1), RN3.2 (R2.1), RN3.3 (R3.1), RN3.4 (R4.1), RN4.1 (R1.1), RN4.2 (R2.1), RN4.3 (R3.1), RN4.4 (R4.1), C28.1, C40.1, C41.1, C42.2, D12.1 (K), H1.1, H2.1, J4.3 (GND), J4.5 (GND), J4.9 (GND), J7.12 (Pin_12), J7.39 (Pin_39), J7.40 (Pin_40), J7.SH (Shield), Q2.3 (E); no longer RN1.5 (R4.2), RN1.6 (R3.2), RN1.7 (R2.2), RN1.8 (R1.2), RN2.5 (R4.2), RN2.6 (R3.2), RN2.7 (R2.2), RN2.8 (R1.2), RN3.5 (R4.2), RN3.6 (R3.2), RN3.7 (R2.2), RN3.8 (R1.2), RN4.5 (R4.2), RN4.6 (R3.2), RN4.7 (R2.2), RN4.8 (R1.2)
- net GPS_3DF: now also U1.86 (PD5)
- net GPS_INT: now also U1.85 (PD4); no longer U1.61 (PD14)
- net LCD_REG_EN: now also U1.60 (PD13); no longer U1.57 (PD10)
- net LTDC_B4: now also RN3.8 (R1.2), J7.16 (Pin_16), J7.20 (Pin_20); no longer RN3.1 (R1.1)
- net LTDC_B5: now also RN3.7 (R2.2), J7.15 (Pin_15), J7.19 (Pin_19); no longer RN3.2 (R2.1)
- net LTDC_B6: now also RN3.6 (R3.2), J7.14 (Pin_14), J7.18 (Pin_18); no longer RN3.3 (R3.1)
- net LTDC_B7: now also RN3.5 (R4.2), J7.13 (Pin_13), J7.17 (Pin_17); no longer RN3.4 (R4.1)
- net LTDC_CK: now also RN4.8 (R1.2), J7.11 (Pin_11); no longer RN4.1 (R1.1)
- net LTDC_DE: now also RN4.7 (R2.2), J7.10 (Pin_10); no longer RN4.2 (R2.1)
- net LTDC_G4: now also RN2.8 (R1.2), J7.24 (Pin_24), J7.28 (Pin_28); no longer RN2.1 (R1.1)
- net LTDC_G5: now also RN2.7 (R2.2), J7.23 (Pin_23), J7.27 (Pin_27); no longer RN2.2 (R2.1)
- net LTDC_G6: now also RN2.6 (R3.2), J7.22 (Pin_22), J7.26 (Pin_26); no longer RN2.3 (R3.1)
- net LTDC_G7: now also RN2.5 (R4.2), J7.21 (Pin_21), J7.25 (Pin_25); no longer RN2.4 (R4.1)
- net LTDC_HS: now also RN4.6 (R3.2), J7.9 (Pin_9); no longer RN4.3 (R3.1)
- net LTDC_R4: now also RN1.8 (R1.2), J7.32 (Pin_32), J7.36 (Pin_36); no longer RN1.1 (R1.1)
- net LTDC_R5: now also RN1.7 (R2.2), U1.68 (PA9), J7.31 (Pin_31), J7.35 (Pin_35); no longer RN1.2 (R2.1), U1.15 (PC0)
- net LTDC_R6: now also RN1.6 (R3.2), J7.30 (Pin_30), J7.34 (Pin_34); no longer RN1.3 (R3.1)
- net LTDC_R7: now also RN1.5 (R4.2), J7.29 (Pin_29), J7.33 (Pin_33); no longer RN1.4 (R4.1)
- net LTDC_VS: now also RN4.5 (R4.2), J7.8 (Pin_8); no longer RN4.4 (R4.1)
- net SPI4_ACCEL_NCS: now also U1.2 (PE3); no longer U1.97 (PE0)
- net STM_STATUS_C: now also U1.18 (PC3_C)
- net STM_STATUS_L: now also U1.15 (PC0); no longer U1.2 (PE3)
- net STM_VCORE_GOOD: now also U1.57 (PD10); no longer U1.60 (PD13)
- net SW_R: no longer U1.18 (PC3_C)
- net TOUCH_INT: no longer U1.88 (PD7)
- net USART3_CTS_NCP: now also U7.21 (P0.07)
- net USART3_RTS_NCP: now also U7.3 (P0.05/AIN3)
- net USART3_RX_NCP: now also U7.20 (P0.08)
- net USART3_TX_NCP: now also U7.2 (P0.06)
- net VCAP1: now also R12.2; no longer R12.1
- net VCAP2: now also R13.2; no longer R13.1
- net VCC_3V3_MCU: now also U2.A4 (RESET#), J4.1 (VCC), J7.37 (Pin_37), J7.38 (Pin_38), R14.1, R21.2; no longer C9.1, R7.2, U11.23 (~RESET), U6.2 (VIN)
- net VCC_CORE: now also R12.1, R13.1; no longer R12.2, R13.2
- net VCC_LCD_PWR: now also C42.1, J7.5 (Pin_5), J7.6 (Pin_6), R15.1
- net VCC_SYS: now also C9.1, U6.2 (VIN)
- net at R84.2: now also J7.1 (Pin_1)
- net at R83.2: now also J7.2 (Pin_2)
- net at R82.2: now also J7.3 (Pin_3)
- net at R20.1, U12.1 (FB): now also J9.4 (Pin_4); no longer J9.1 (Pin_1)
- net NCP_STATUS_0: now reaches U7.15 (NFC/P0.10)
- net NCP_STATUS_0: now also R22.1
- net PD15_NCP: now reaches U7.24 (P0.28/AIN4)
- net PD15_NCP: now also U1.62 (PD15)
- net at U7.4 (P0.00/XL1): now also C41.2, Y2.2
- net at U7.5 (P0.01/XL2): now also C40.2, Y2.1
- net at U7.7 (DEC4): now also C28.2
- net GPS_FORCE_ON renamed GPS_FORCEON
- net GPS_FORCEON: no longer U1.62 (PD15)
- net LPUART1_RX_GPS renamed BUZZER_T1C3
- net BUZZER_T1C3: no longer U11.25 (TXD1)
- net LPUART1_TX_GPS renamed GPS_UART8_TX
- net GPS_UART8_TX: no longer U1.68 (PA9)
- net SD_VSEL: no longer names the net of U1.82 (PD1)
- new net: BZ1.1 (-), R14.2, R15.2, R7.2
- new net: BZ1.2 (+), Q2.2 (C), R7.1
- new net: D12.2 (A), R22.2
- new net BUZZER_PWM: Q2.1 (B)
- new net GPS_UART8_RX: U1.97 (PE0), U11.25 (TXD1)
- new net PD14_NCP: U1.61 (PD14), U7.25 (P0.20/TRACECLK)
- no-connect marks 11 -> 15
Other:
- moved on the sheet: C15, C16, C17, C2, C30, C38, C46, C50, C59, C61, C63, C65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

Commit message: silkscreen
Parts:
- added L6: 10u, Inductor_SMD:L_Wuerth_MAPI-2510, symbol Device:L_Small
- added N1: Bottom Silk Art, atlas:europeart, symbol Mechanical:Housing
- H1, H2, H3, H4: footprint MountingHole:MountingHole_2.7mm_M2.5_Pad_Via -> MountingHole:MountingHole_2.2mm_M2_Pad_Via
Connections:
- net VCC_3V3_MCU: no longer SW7.1
- net VCC_BACKUP: now also SW7.1
- net at C28.2, U7.7 (DEC4): now also L6.1
- net at C41.2, U7.4 (P0.00/XL1): now also Y2.1; no longer Y2.2
- net at C40.2, U7.5 (P0.01/XL2): now also Y2.2; no longer Y2.1
- net at U7.6 (DCC): now also L6.2
- no-connect marks 15 -> 14
Other:
- moved on the sheet: D10, D12, D5, D8, R11, R18, R19, R22

Commit message: PCB to fab
Parts:
- added R10, R17: 100k, Resistor_SMD:R_0603_1608Metric, symbol Device:R_Small
- added R16: NP, Resistor_SMD:R_0603_1608Metric, symbol Device:R_Small
- added R23: 0, Jumper:SolderJumper-2_P1.3mm_Open_TrianglePad1.0x1.5mm, symbol Device:R_Small
- added R24, R30: NP, Jumper:SolderJumper-2_P1.3mm_Open_TrianglePad1.0x1.5mm, symbol Device:R_Small
- added R31: 0, Resistor_SMD:R_0402_1005Metric, symbol Device:R_Small
- added TP1: 5V_USB, TestPoint:TestPoint_THTPad_D1.0mm_Drill0.5mm, symbol Connector:TestPoint
- added TP10: LCD_BL, TestPoint:TestPoint_THTPad_D1.0mm_Drill0.5mm, symbol Connector:TestPoint
- added TP11, TP12: GND, TestPoint:TestPoint_THTPad_D1.0mm_Drill0.5mm, symbol Connector:TestPoint
- added TP13: VSYS, TestPoint:TestPoint_THTPad_D1.0mm_Drill0.5mm, symbol Connector:TestPoint
- added TP2: 3V_BACKUP, TestPoint:TestPoint_THTPad_D1.0mm_Drill0.5mm, symbol Connector:TestPoint
- added TP3: 3V3_MCU, TestPoint:TestPoint_THTPad_D1.0mm_Drill0.5mm, symbol Connector:TestPoint
- added TP4: SCL, TestPoint:TestPoint_THTPad_D1.0mm_Drill0.5mm, symbol Connector:TestPoint
- added TP5: SDA, TestPoint:TestPoint_THTPad_D1.0mm_Drill0.5mm, symbol Connector:TestPoint
- added TP6: SCLK, TestPoint:TestPoint_THTPad_D1.0mm_Drill0.5mm, symbol Connector:TestPoint
- added TP7: MOSI, TestPoint:TestPoint_THTPad_D1.0mm_Drill0.5mm, symbol Connector:TestPoint
- added TP8: MISO, TestPoint:TestPoint_THTPad_D1.0mm_Drill0.5mm, symbol Connector:TestPoint
- added TP9: LCD_5V, TestPoint:TestPoint_THTPad_D1.0mm_Drill0.5mm, symbol Connector:TestPoint
- Q2: value Q_NPN_BCE -> BC817K; symbol Device:Q_NPN_BCE -> Device:Q_NPN_BEC
Connections:
- net BUZZER_PWM is gone; now on net BUZZER_T1C3: Q2.1 (B)
- net BL_HV: now also TP10.1
- net GND: now also J3.3 (Pin_3), Q2.2 (E), R10.1, TP11.1, TP12.1; no longer J3.5 (Pin_5), Q2.3 (E)
- net GPS_FORCEON: now also U1.82 (PD1); no longer U1.95 (PB8)
- net I2C4_SCL_SENSOR: now also J3.6 (Pin_6), TP4.1; no longer J3.1 (Pin_1)
- net I2C4_SDA_SENSOR: now also J3.5 (Pin_5), TP5.1; no longer J3.2 (Pin_2)
- net MCU_3V3_EN: now also R16.1, R17.1
- net SPI4_MISO_APP: now also TP8.1
- net SPI4_MOSI_APP: now also TP7.1
- net SPI4_SCK_APP: now also TP6.1
- net STM_VCORE_EN: now also R10.2
- net TOUCH_INT: now also J3.4 (Pin_4); no longer J3.3 (Pin_3)
- net USB_CHG_D+: now also R41.1; no longer R43.1
- net USB_CHG_D-: now also R43.1; no longer R41.1
- net USB_PORT_D+: now also R41.2; no longer R43.2
- net USB_PORT_D-: now also R43.2; no longer R41.2
- net USB_PORT_VBUS: now also TP1.1
- net VCC_3V3_MCU: now also J3.2 (Pin_2), R17.2, R24.1, TP3.1; no longer J3.4 (Pin_4), U2.A4 (RESET#)
- net VCC_BACKUP: now also R16.2, TP2.1
- net VCC_LCD_PWR: now also R23.1; no longer C42.1, C53.1, J7.5 (Pin_5), J7.6 (Pin_6)
- net VCC_SYS: now also R30.1, TP13.1
- net at J7.1 (Pin_1), R84.2: now also R31.1
- net at BZ1.2 (+), R7.1: now also Q2.3 (C); no longer Q2.2 (C)
- net at R3.2: now also J3.1 (Pin_1); no longer J3.6 (Pin_6)
- new net: C42.1, C53.1, J7.5 (Pin_5), J7.6 (Pin_6), R23.2, R24.2, R30.2, TP9.1
- new net LCD_OPT: R31.2, U1.95 (PB8)
- no-connect marks 14 -> 15
Other:
- moved on the sheet: C20, C30, C38, C42, C46, C53, C54, C9, J3, J7, R28, R29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
